File: hw/ZakladniElektronika/HlavniDeska/ESP332S3.kicad_sch (KiCad schematic)
At the start: 11 parts, among them J1 ESP-Programing_conector, U10 ESP32-S3-WROOM

Commit message: WIP
Parts:
- C132, C133: Basic/Extended (none) -> E; LCSC C52923 -> C1518208; info (none) -> 50V, X7R
- C135: Basic/Extended (none) -> B; JLCPCB_CORRECTION 0;0;0 -> (none); LCSC C1525 -> C307331; info (none) -> 50V, X7R
Changed lines of the file:
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@@
     (effects (font (size 1.27 1.27)) (justify left))
   )
-  (hierarchical_label "BOOT" (shape bidirectional) (at 153.67 69.85 180) (fields_autoplaced)
+  (hierarchical_label "BOOT" (shape input) (at 153.67 69.85 180) (fields_autoplaced)
     (effects (font (size 1.27 1.27)) (justify right))
   )
@@
       (effects (font (size 1.27 1.27)) hide)
     )
-    (property "LCSC" "C52923" (at 195.58 87.63 0)
+    (property "LCSC" "C1518208" (at 195.58 87.63 0)
       (effects (font (size 1.27 1.27)) hide)
     )
     (property "JLCPCB_CORRECTION" "0;0;0" (at 195.58 87.63 0)
+      (effects (font (size 1.27 1.27)) hide)
+    )
+    (property "Basic/Extended" "E" (at 195.58 87.63 0)
+      (effects (font (size 1.27 1.27)) hide)
+    )
+    (property "info" "50V, X7R" (at 195.58 87.63 0)
       (effects (font (size 1.27 1.27)) hide)
     )
@@
       (effects (font (size 1.27 1.27)) hide)
     )
-    (property "LCSC" "C52923" (at 180.34 87.63 0)
+    (property "LCSC" "C1518208" (at 180.34 87.63 0)
       (effects (font (size 1.27 1.27)) hide)
     )
     (property "JLCPCB_CORRECTION" "0;0;0" (at 180.34 87.63 0)
+      (effects (font (size 1.27 1.27)) hide)
+    )
+    (property "Basic/Extended" "E" (at 180.34 87.63 0)
+      (effects (font (size 1.27 1.27)) hide)
+    )
+    (property "info" "50V, X7R" (at 180.34 87.63 0)
       (effects (font (size 1.27 1.27)) hide)
     )
@@
       (effects (font (size 1.27 1.27)) hide)
     )
-    (property "LCSC" "C1525" (at 218.44 43.18 0)
-      (effects (font (size 1.27 1.27)) hide)
-    )
-    (property "JLCPCB_CORRECTION" "0;0;0" (at 218.44 43.18 0)
-      (effects (font (size 1.27 1.27)) hide)
-    )
+    (property "LCSC" "C307331" (at 218.44 43.18 0)
+      (effects (font (size 1.27 1.27)) hide)
+    )
+    (property "JLCPCB_CORRECTION" "" (at 218.44 43.18 0)
+      (effects (font (size 1.27 1.27)) hide)
+    )
+    (property "Basic/Extended" "B" (at 218.44 43.18 0)
+      (effects (font (size 1.27 1.27)) hide)
+    )
+    (property "info" "50V, X7R" (at 218.44 43.18 0)
+      (effects (font (size 1.27 1.27)) hide)
+    )

Commit message: Nastin schematu
Connections:
- net EN renamed RST
Other:
- moved on the sheet: J1
Changed lines of the file:
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@@
     (stroke (width 0.25) (type default))
   )
-  (wire (pts (xy 57.15 69.85) (xy 54.61 69.85))
-    (stroke (width 0) (type default))
-  )
-  (wire (pts (xy 52.07 77.47) (xy 57.15 77.47))
+  (wire (pts (xy 60.96 81.28) (xy 58.42 81.28))
+    (stroke (width 0) (type default))
+  )
+  (wire (pts (xy 55.88 88.9) (xy 60.96 88.9))
     (stroke (width 0) (type default))
   )
@@
     (stroke (width 0.53) (type default))
   )
-  (wire (pts (xy 54.61 69.85) (xy 54.61 67.31))
+  (wire (pts (xy 58.42 81.28) (xy 58.42 78.74))
     (stroke (width 0) (type default))
   )
@@
     (stroke (width 0) (type default))
   )
-  (wire (pts (xy 52.07 74.93) (xy 57.15 74.93))
+  (wire (pts (xy 55.88 86.36) (xy 60.96 86.36))
     (stroke (width 0) (type default))
   )
@@
     (stroke (width 0) (type default))
   )
-  (wire (pts (xy 54.61 72.39) (xy 57.15 72.39))
+  (wire (pts (xy 58.42 83.82) (xy 60.96 83.82))
     (stroke (width 0) (type default))
   )
@@
     (stroke (width 0) (type default))
   )
-  (wire (pts (xy 52.07 80.01) (xy 57.15 80.01))
+  (wire (pts (xy 55.88 91.44) (xy 60.96 91.44))
     (stroke (width 0) (type default))
   )
@@
     (stroke (width 0) (type default))
   )
-  (wire (pts (xy 52.07 82.55) (xy 57.15 82.55))
+  (wire (pts (xy 55.88 93.98) (xy 60.96 93.98))
     (stroke (width 0) (type default))
   )
@@
     (stroke (width 0) (type default))
   )
-  (wire (pts (xy 54.61 85.09) (xy 54.61 72.39))
+  (wire (pts (xy 58.42 96.52) (xy 58.42 83.82))
     (stroke (width 0) (type default))
   )
@@
     (stroke (width 0) (type default))
   )
-  (wire (pts (xy 187.96 58.42) (xy 195.58 58.42))
+  (wire (pts (xy 193.04 58.42) (xy 195.58 58.42))
     (stroke (width 0) (type default))
   )
@@
     (effects (font (size 1.27 1.27)) (justify right bottom))
   )
-  (label "EN" (at 52.07 74.93 180) (fields_autoplaced)
+  (label "EN" (at 55.88 86.36 180) (fields_autoplaced)
     (effects (font (size 1.27 1.27)) (justify right bottom))
   )
-  (label "RX0" (at 52.07 80.01 180) (fields_autoplaced)
+  (label "RX0" (at 55.88 91.44 180) (fields_autoplaced)
     (effects (font (size 1.27 1.27)) (justify right bottom))
   )
-  (label "TX0" (at 52.07 82.55 180) (fields_autoplaced)
+  (label "TX0" (at 55.88 93.98 180) (fields_autoplaced)
     (effects (font (size 1.27 1.27)) (justify right bottom))
   )
-  (label "EN" (at 187.96 58.42 0) (fields_autoplaced)
+  (label "EN" (at 196.85 58.42 0) (fields_autoplaced)
     (effects (font (size 1.27 1.27)) (justify left bottom))
   )
-  (label "BOOT" (at 52.07 77.47 180) (fields_autoplaced)
+  (label "BOOT" (at 55.88 88.9 180) (fields_autoplaced)
     (effects (font (size 1.27 1.27)) (justify right bottom))
   )
@@
   (hierarchical_label "3V3" (shape input) (at 180.34 59.69 90) (fields_autoplaced)
     (effects (font (size 1.27 1.27)) (justify left))
+  )
+  (hierarchical_label "RST" (shape input) (at 193.04 58.42 180) (fields_autoplaced)
+    (effects (font (size 1.27 1.27)) (justify right))
   )
   (hierarchical_label "GND" (shape input) (at 162.56 91.44 270) (fields_autoplaced)
@@
     )
   )
-  (symbol (lib_id "power:GND") (at 54.61 85.09 0) (unit 1)
+  (symbol (lib_id "power:GND") (at 58.42 96.52 0) (unit 1)
     (in_bom yes) (on_board yes) (dnp no) (fields_autoplaced)
-    (property "Reference" "#PWR02" (at 54.61 91.44 0)
-      (effects (font (size 1.27 1.27)) hide)
-    )
-    (property "Value" "GND" (at 54.61 90.17 0)
+    (property "Reference" "#PWR02" (at 58.42 102.87 0)
+      (effects (font (size 1.27 1.27)) hide)
+    )
+    (property "Value" "GND" (at 58.42 101.6 0)
       (effects (font (size 1.27 1.27)))
     )
-    (property "Footprint" "" (at 54.61 85.09 0)
-      (effects (font (size 1.27 1.27)) hide)
-    )
-    (property "Datasheet" "" (at 54.61 85.09 0)
+    (property "Footprint" "" (at 58.42 96.52 0)
+      (effects (font (size 1.27 1.27)) hide)
+    )
+    (property "Datasheet" "" (at 58.42 96.52 0)
       (effects (font (size 1.27 1.27)) hide)
     )
@@
     )
   )
-  (symbol (lib_id "power:+5V") (at 54.61 67.31 0) (mirror y) (unit 1)
+  (symbol (lib_id "power:+5V") (at 58.42 78.74 0) (mirror y) (unit 1)
     (in_bom yes) (on_board yes) (dnp no) (fields_autoplaced)
-    (property "Reference" "#PWR01" (at 54.61 71.12 0)
-      (effects (font (size 1.27 1.27)) hide)
-    )
-    (property "Value" "+5V" (at 54.61 62.23 0)
+    (property "Reference" "#PWR01" (at 58.42 82.55 0)
+      (effects (font (size 1.27 1.27)) hide)
+    )
+    (property "Value" "+5V" (at 58.42 73.66 0)
       (effects (font (size 1.27 1.27)))
     )
-    (property "Footprint" "" (at 54.61 67.31 0)
-      (effects (font (size 1.27 1.27)) hide)
-    )
-    (property "Datasheet" "" (at 54.61 67.31 0)
+    (property "Footprint" "" (at 58.42 78.74 0)
+      (effects (font (size 1.27 1.27)) hide)
+    )
+    (property "Datasheet" "" (at 58.42 78.74 0)
       (effects (font (size 1.27 1.27)) hide)
     )
@@
     )
   )
-  (symbol (lib_id "Robotarna_KiCad_Library:ESP-Programing_conector") (at 62.23 69.85 0) (unit 1)
-    (in_bom yes) (on_board yes) (dnp no)
-    (property "Reference" "J1" (at 59.69 63.5 0)
-      (effects (font (size 1.27 1.27)) (justify left))
-    )
-    (property "Value" "ESP-Programing_conector" (at 59.69 66.04 0)
-      (effects (font (size 1.27 1.27)) (justify left))
-    )
-    (property "Footprint" "Robotarna_KiCad_Library:ESP-Programing_conector" (at 62.23 67.31 0)
-      (effects (font (size 1.27 1.27)) hide)
-    )
-    (property "Datasheet" "" (at 62.23 69.85 0)
-      (effects (font (size 1.27 1.27)) hide)
-    )
+  (symbol (lib_id "Robotarna_KiCad_Library:ESP-Programing_conector") (at 66.04 81.28 0) (unit 1)
+    (in_bom yes) (on_board yes) (dnp no)
+    (property "Reference" "J1" (at 63.5 74.93 0)
+      (effects (font (size 1.27 1.27)) (justify left))
+    )
+    (property "Value" "ESP-Programing_conector" (at 63.5 77.47 0)
+      (effects (font (size 1.27 1.27)) (justify left))
+    )
+    (property "Footprint" "Robotarna_KiCad_Library:ESP-Programing_conector" (at 66.04 78.74 0)
+      (effects (font (size 1.27 1.27)) hide)
+    )
+    (property "Datasheet" "" (at 66.04 81.28 0)
+      (effects (font (size 1.27 1.27)) hide)
+    )

Commit message: Zaciame psat
Parts:
- added D1: ${SIM.PARAMS}, Diode_SMD:D_SMA, symbol Device:D
Connections:
- net +5V: no longer names the net of J1.1 (VCC)
- net +5V: now also D1.2 (A)
- new net 5V-(programator): D1.1 (K)
Changed lines of the file:
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@@
     (stroke (width 0.25) (type default))
   )
-  (wire (pts (xy 60.96 81.28) (xy 58.42 81.28))
+  (wire (pts (xy 60.96 81.28) (xy 53.34 81.28))
     (stroke (width 0) (type default))
   )
@@
     (stroke (width 0.53) (type default))
   )
-  (wire (pts (xy 58.42 81.28) (xy 58.42 78.74))
+  (wire (pts (xy 53.34 81.28) (xy 53.34 78.74))
     (stroke (width 0) (type default))
   )
@@
     (effects (font (size 1.27 1.27)) (justify right))
   )
+  (hierarchical_label "GND" (shape input) (at 58.42 96.52 270) (fields_autoplaced)
+    (effects (font (size 1.27 1.27)) (justify right))
+  )
   (hierarchical_label "IO15" (shape bidirectional) (at 234.95 88.9 0) (fields_autoplaced)
     (effects (font (size 1.27 1.27)) (justify left))
@@
   )
   (hierarchical_label "IO17" (shape bidirectional) (at 234.95 93.98 0) (fields_autoplaced)
+    (effects (font (size 1.27 1.27)) (justify left))
+  )
+  (hierarchical_label "5V-(programator)" (shape input) (at 53.34 71.12 90) (fields_autoplaced)
     (effects (font (size 1.27 1.27)) (justify left))
   )
@@
     )
   )
-  (symbol (lib_id "power:GND") (at 58.42 96.52 0) (unit 1)
-    (in_bom yes) (on_board yes) (dnp no) (fields_autoplaced)
-    (property "Reference" "#PWR02" (at 58.42 102.87 0)
-      (effects (font (size 1.27 1.27)) hide)
-    )
-    (property "Value" "GND" (at 58.42 101.6 0)
-      (effects (font (size 1.27 1.27)))
-    )
-    (property "Footprint" "" (at 58.42 96.52 0)
-      (effects (font (size 1.27 1.27)) hide)
-    )
-    (property "Datasheet" "" (at 58.42 96.52 0)
-      (effects (font (size 1.27 1.27)) hide)
-    )
-    (pin "1")
-    (instances
-      (project "ZakladniElektronika"
-        (path "/99cd3e15-4eb6-4cbb-8726-789aedd3df15/c3b70d9b-0dcb-4344-9507-13ff5b4c000e/3abb0ef0-3dd5-4818-a187-7e9bc43bafd4"
-          (reference "#PWR02") (unit 1)
-        )
-      )
-      (project "SemiSemafor"
-        (path "/fb82d987-26cf-425e-8e99-22ecb59c8a96"
-          (reference "#PWR0112") (unit 1)
-        )
-      )
-    )
-  )
-  (symbol (lib_id "power:+5V") (at 58.42 78.74 0) (mirror y) (unit 1)
-    (in_bom yes) (on_board yes) (dnp no) (fields_autoplaced)
-    (property "Reference" "#PWR01" (at 58.42 82.55 0)
-      (effects (font (size 1.27 1.27)) hide)
-    )
-    (property "Value" "+5V" (at 58.42 73.66 0)
-      (effects (font (size 1.27 1.27)))
-    )
-    (property "Footprint" "" (at 58.42 78.74 0)
-      (effects (font (size 1.27 1.27)) hide)
-    )
-    (property "Datasheet" "" (at 58.42 78.74 0)
-      (effects (font (size 1.27 1.27)) hide)
-    )
-    (pin "1")
-    (instances
-      (project "ZakladniElektronika"
-        (path "/99cd3e15-4eb6-4cbb-8726-789aedd3df15/c3b70d9b-0dcb-4344-9507-13ff5b4c000e/3abb0ef0-3dd5-4818-a187-7e9bc43bafd4"
-          (reference "#PWR01") (unit 1)
-        )
-      )
-      (project "SemiSemafor"
-        (path "/fb82d987-26cf-425e-8e99-22ecb59c8a96"
-          (reference "#PWR0129") (unit 1)
-        )
-      )
-    )
-  )
   (symbol (lib_id "Device:R") (at 195.58 50.8 0) (unit 1)
     (in_bom yes) (on_board yes) (dnp no)
@@
         )
       )
+    )
+  )
+  (symbol (lib_id "Device:D") (at 53.34 74.93 90) (mirror x) (unit 1)
+    (in_bom yes) (on_board yes) (dnp no)
+    (property "Reference" "D1" (at 48.26 74.93 90)
+      (effects (font (size 1.27 1.27)))
+    )
+    (property "Value" "${SIM.PARAMS}" (at 50.8 74.93 0)
+      (effects (font (size 1.27 1.27)) hide)
+    )
+    (property "Footprint" "Diode_SMD:D_SMA" (at 53.34 74.93 0)
+      (effects (font (size 1.27 1.27)) hide)
+    )
+    (property "Datasheet" "~" (at 53.34 74.93 0)
+      (effects (font (size 1.27 1.27)) hide)
+    )
+    (property "LCSC" "C8678" (at 53.34 74.93 0)
+      (effects (font (size 1.27 1.27)) hide)
+    )
+    (property "JLCPCB_CORRECTION" "0;0;0" (at 53.34 74.93 0)
+      (effects (font (size 1.27 1.27)) hide)
+    )
+    (property "Sim.Device" "SPICE" (at 53.34 74.93 0)
+      (effects (font (size 1.27 1.27)) (justify left) hide)
+    )
+    (property "Sim.Params" "type=\"D\" model=\"DIODE\" lib=\"\"" (at 5.08 142.24 0)
+      (effects (font (size 1.27 1.27)) hide)
+    )
+    (property "Sim.Pins" "1=1 2=2" (at 5.08 142.24 0)
+      (effects (font (size 1.27 1.27)) hide)
+    )
+    (pin "1")
+    (pin "2")
+    (instances
+      (project "ESP32xx_programmer"
+        (path "/0ff82e5d-9817-4600-b531-27674345b32d"
+          (reference "D1") (unit 1)
+        )
+      )
+      (project "ZakladniElektronika"
+        (path "/99cd3e15-4eb6-4cbb-8726-789aedd3df15/c3b70d9b-0dcb-4344-9507-13ff5b4c000e/3abb0ef0-3dd5-4818-a187-7e9bc43bafd4"
+          (reference "D121") (unit 1)
+        )
+      )
