File: hw/ZakladniElektronika/HlavniDeska/PNU.kicad_sch (KiCad schematic)
At the start: 2 parts, among them Q6 Q_NMOS_DGS

Commit message: Nastin schematu
Parts:
- renumbered Q6 to Q8, R19 to R2
Other:
- note added: "Prevodnik Napetovich Urovni(PNU)"
- note removed: "Prevodnik Napetovich Urovni(PNU) invertujici"
Changed lines of the file:
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@@
     (stroke (width 0) (type default))
   )
-  (text "Prevodnik Napetovich Urovni(PNU) invertujici" (at 73.66 27.94 0)
+  (text "Prevodnik Napetovich Urovni(PNU)" (at 83.82 25.4 0)
     (effects (font (size 2 2)) (justify left bottom))
   )
@@
   (symbol (lib_id "Device:Q_NMOS_DGS") (at 107.95 62.23 90) (mirror x) (unit 1)
     (in_bom yes) (on_board yes) (dnp no)
-    (property "Reference" "Q6" (at 109.22 71.12 90)
+    (property "Reference" "Q8" (at 109.22 71.12 90)
       (effects (font (size 1.27 1.27)) (justify left))
     )
@@
     (instances
       (project "ZakladniElektronika"
-        (path "/99cd3e15-4eb6-4cbb-8726-789aedd3df15/c3b70d9b-0dcb-4344-9507-13ff5b4c000e/2d5c8383-b4dd-4e50-a76e-5d9de1ae531a/eab0e57f-22d7-4e2c-8f9b-b1863d6f54c5"
-          (reference "Q2") (unit 1)
-        )
-        (path "/99cd3e15-4eb6-4cbb-8726-789aedd3df15/c3b70d9b-0dcb-4344-9507-13ff5b4c000e/2d5c8383-b4dd-4e50-a76e-5d9de1ae531a"
-          (reference "Q9") (unit 1)
-        )
-        (path "/99cd3e15-4eb6-4cbb-8726-789aedd3df15/c3b70d9b-0dcb-4344-9507-13ff5b4c000e/2d5c8383-b4dd-4e50-a76e-5d9de1ae531a/6f15d501-5fa4-4bfe-a53d-adacae284de5"
-          (reference "Q3") (unit 1)
-        )
         (path "/99cd3e15-4eb6-4cbb-8726-789aedd3df15/c3b70d9b-0dcb-4344-9507-13ff5b4c000e/2d5c8383-b4dd-4e50-a76e-5d9de1ae531a/4fe93ea1-faa6-4fe1-9624-81c4f018fba5"
           (reference "Q8") (unit 1)
@@
           (reference "Q6") (unit 1)
         )
+        (path "/99cd3e15-4eb6-4cbb-8726-789aedd3df15/c3b70d9b-0dcb-4344-9507-13ff5b4c000e/2d5c8383-b4dd-4e50-a76e-5d9de1ae531a/eab0e57f-22d7-4e2c-8f9b-b1863d6f54c5"
+          (reference "Q2") (unit 1)
+        )
+        (path "/99cd3e15-4eb6-4cbb-8726-789aedd3df15/c3b70d9b-0dcb-4344-9507-13ff5b4c000e/2d5c8383-b4dd-4e50-a76e-5d9de1ae531a"
+          (reference "Q9") (unit 1)
+        )
+        (path "/99cd3e15-4eb6-4cbb-8726-789aedd3df15/c3b70d9b-0dcb-4344-9507-13ff5b4c000e/2d5c8383-b4dd-4e50-a76e-5d9de1ae531a/6f15d501-5fa4-4bfe-a53d-adacae284de5"
+          (reference "Q3") (unit 1)
+        )
       )
       (project "Zdroj"
@@
   (symbol (lib_id "Device:R") (at 115.57 48.26 0) (unit 1)
     (in_bom yes) (on_board yes) (dnp no)
-    (property "Reference" "R19" (at 118.11 46.99 0)
+    (property "Reference" "R2" (at 118.11 46.99 0)
       (effects (font (size 1.27 1.27)) (justify left))
     )
@@
     (instances
       (project "ZakladniElektronika"
-        (path "/99cd3e15-4eb6-4cbb-8726-789aedd3df15/c3b70d9b-0dcb-4344-9507-13ff5b4c000e/2d5c8383-b4dd-4e50-a76e-5d9de1ae531a/4fe93ea1-faa6-4fe1-9624-81c4f018fba5"
-          (reference "R19") (unit 1)
+        (path "/99cd3e15-4eb6-4cbb-8726-789aedd3df15/c3b70d9b-0dcb-4344-9507-13ff5b4c000e/2d5c8383-b4dd-4e50-a76e-5d9de1ae531a/eab0e57f-22d7-4e2c-8f9b-b1863d6f54c5"
+          (reference "R2") (unit 1)
+        )
+        (path "/99cd3e15-4eb6-4cbb-8726-789aedd3df15/c3b70d9b-0dcb-4344-9507-13ff5b4c000e/2d5c8383-b4dd-4e50-a76e-5d9de1ae531a"
+          (reference "R35") (unit 1)
+        )
+        (path "/99cd3e15-4eb6-4cbb-8726-789aedd3df15/c3b70d9b-0dcb-4344-9507-13ff5b4c000e/3abb0ef0-3dd5-4818-a187-7e9bc43bafd4"
+          (reference "R8") (unit 1)
+        )
+        (path "/99cd3e15-4eb6-4cbb-8726-789aedd3df15/c3b70d9b-0dcb-4344-9507-13ff5b4c000e/2d5c8383-b4dd-4e50-a76e-5d9de1ae531a/6f15d501-5fa4-4bfe-a53d-adacae284de5"
+          (reference "R14") (unit 1)
         )
         (path "/99cd3e15-4eb6-4cbb-8726-789aedd3df15/c3b70d9b-0dcb-4344-9507-13ff5b4c000e/2d5c8383-b4dd-4e50-a76e-5d9de1ae531a/b0eb48ce-ce27-474b-a2c8-9099028688a0"
           (reference "R20") (unit 1)
+        )
+        (path "/99cd3e15-4eb6-4cbb-8726-789aedd3df15/c3b70d9b-0dcb-4344-9507-13ff5b4c000e/2d5c8383-b4dd-4e50-a76e-5d9de1ae531a/4fe93ea1-faa6-4fe1-9624-81c4f018fba5"
+          (reference "R19") (unit 1)
         )
         (path "/99cd3e15-4eb6-4cbb-8726-789aedd3df15/c3b70d9b-0dcb-4344-9507-13ff5b4c000e/2d5c8383-b4dd-4e50-a76e-5d9de1ae531a/1491371a-c228-41d9-8946-b539dbebb3b9"
@@
           (reference "R17") (unit 1)
         )
-        (path "/99cd3e15-4eb6-4cbb-8726-789aedd3df15/c3b70d9b-0dcb-4344-9507-13ff5b4c000e/2d5c8383-b4dd-4e50-a76e-5d9de1ae531a/eab0e57f-22d7-4e2c-8f9b-b1863d6f54c5"
-          (reference "R2") (unit 1)
-        )
-        (path "/99cd3e15-4eb6-4cbb-8726-789aedd3df15/c3b70d9b-0dcb-4344-9507-13ff5b4c000e/2d5c8383-b4dd-4e50-a76e-5d9de1ae531a"
-          (reference "R35") (unit 1)
-        )
-        (path "/99cd3e15-4eb6-4cbb-8726-789aedd3df15/c3b70d9b-0dcb-4344-9507-13ff5b4c000e/3abb0ef0-3dd5-4818-a187-7e9bc43bafd4"
-          (reference "R8") (unit 1)
-        )
-        (path "/99cd3e15-4eb6-4cbb-8726-789aedd3df15/c3b70d9b-0dcb-4344-9507-13ff5b4c000e/2d5c8383-b4dd-4e50-a76e-5d9de1ae531a/6f15d501-5fa4-4bfe-a53d-adacae284de5"
-          (reference "R14") (unit 1)
-        )
       )

Commit message: Zaciame psat
Parts:
- renumbered Q8 to Q2, R2 to R19
Changed lines of the file:
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@@
   (symbol (lib_id "Device:Q_NMOS_DGS") (at 107.95 62.23 90) (mirror x) (unit 1)
     (in_bom yes) (on_board yes) (dnp no)
-    (property "Reference" "Q8" (at 109.22 71.12 90)
+    (property "Reference" "Q2" (at 109.22 71.12 90)
       (effects (font (size 1.27 1.27)) (justify left))
     )
@@
     (instances
       (project "ZakladniElektronika"
+        (path "/99cd3e15-4eb6-4cbb-8726-789aedd3df15/c3b70d9b-0dcb-4344-9507-13ff5b4c000e/2d5c8383-b4dd-4e50-a76e-5d9de1ae531a/eab0e57f-22d7-4e2c-8f9b-b1863d6f54c5"
+          (reference "Q2") (unit 1)
+        )
+        (path "/99cd3e15-4eb6-4cbb-8726-789aedd3df15/c3b70d9b-0dcb-4344-9507-13ff5b4c000e/2d5c8383-b4dd-4e50-a76e-5d9de1ae531a"
+          (reference "Q9") (unit 1)
+        )
+        (path "/99cd3e15-4eb6-4cbb-8726-789aedd3df15/c3b70d9b-0dcb-4344-9507-13ff5b4c000e/2d5c8383-b4dd-4e50-a76e-5d9de1ae531a/6f15d501-5fa4-4bfe-a53d-adacae284de5"
+          (reference "Q3") (unit 1)
+        )
         (path "/99cd3e15-4eb6-4cbb-8726-789aedd3df15/c3b70d9b-0dcb-4344-9507-13ff5b4c000e/2d5c8383-b4dd-4e50-a76e-5d9de1ae531a/4fe93ea1-faa6-4fe1-9624-81c4f018fba5"
           (reference "Q8") (unit 1)
@@
           (reference "Q6") (unit 1)
         )
-        (path "/99cd3e15-4eb6-4cbb-8726-789aedd3df15/c3b70d9b-0dcb-4344-9507-13ff5b4c000e/2d5c8383-b4dd-4e50-a76e-5d9de1ae531a/eab0e57f-22d7-4e2c-8f9b-b1863d6f54c5"
-          (reference "Q2") (unit 1)
-        )
-        (path "/99cd3e15-4eb6-4cbb-8726-789aedd3df15/c3b70d9b-0dcb-4344-9507-13ff5b4c000e/2d5c8383-b4dd-4e50-a76e-5d9de1ae531a"
-          (reference "Q9") (unit 1)
-        )
-        (path "/99cd3e15-4eb6-4cbb-8726-789aedd3df15/c3b70d9b-0dcb-4344-9507-13ff5b4c000e/2d5c8383-b4dd-4e50-a76e-5d9de1ae531a/6f15d501-5fa4-4bfe-a53d-adacae284de5"
-          (reference "Q3") (unit 1)
-        )
       )
       (project "Zdroj"
@@
   (symbol (lib_id "Device:R") (at 115.57 48.26 0) (unit 1)
     (in_bom yes) (on_board yes) (dnp no)
-    (property "Reference" "R2" (at 118.11 46.99 0)
+    (property "Reference" "R19" (at 118.11 46.99 0)
       (effects (font (size 1.27 1.27)) (justify left))
     )
@@
     (instances
       (project "ZakladniElektronika"
-        (path "/99cd3e15-4eb6-4cbb-8726-789aedd3df15/c3b70d9b-0dcb-4344-9507-13ff5b4c000e/2d5c8383-b4dd-4e50-a76e-5d9de1ae531a/eab0e57f-22d7-4e2c-8f9b-b1863d6f54c5"
-          (reference "R2") (unit 1)
-        )
-        (path "/99cd3e15-4eb6-4cbb-8726-789aedd3df15/c3b70d9b-0dcb-4344-9507-13ff5b4c000e/2d5c8383-b4dd-4e50-a76e-5d9de1ae531a"
-          (reference "R35") (unit 1)
-        )
-        (path "/99cd3e15-4eb6-4cbb-8726-789aedd3df15/c3b70d9b-0dcb-4344-9507-13ff5b4c000e/3abb0ef0-3dd5-4818-a187-7e9bc43bafd4"
-          (reference "R8") (unit 1)
-        )
-        (path "/99cd3e15-4eb6-4cbb-8726-789aedd3df15/c3b70d9b-0dcb-4344-9507-13ff5b4c000e/2d5c8383-b4dd-4e50-a76e-5d9de1ae531a/6f15d501-5fa4-4bfe-a53d-adacae284de5"
-          (reference "R14") (unit 1)
+        (path "/99cd3e15-4eb6-4cbb-8726-789aedd3df15/c3b70d9b-0dcb-4344-9507-13ff5b4c000e/2d5c8383-b4dd-4e50-a76e-5d9de1ae531a/4fe93ea1-faa6-4fe1-9624-81c4f018fba5"
+          (reference "R19") (unit 1)
         )
         (path "/99cd3e15-4eb6-4cbb-8726-789aedd3df15/c3b70d9b-0dcb-4344-9507-13ff5b4c000e/2d5c8383-b4dd-4e50-a76e-5d9de1ae531a/b0eb48ce-ce27-474b-a2c8-9099028688a0"
           (reference "R20") (unit 1)
-        )
-        (path "/99cd3e15-4eb6-4cbb-8726-789aedd3df15/c3b70d9b-0dcb-4344-9507-13ff5b4c000e/2d5c8383-b4dd-4e50-a76e-5d9de1ae531a/4fe93ea1-faa6-4fe1-9624-81c4f018fba5"
-          (reference "R19") (unit 1)
         )
         (path "/99cd3e15-4eb6-4cbb-8726-789aedd3df15/c3b70d9b-0dcb-4344-9507-13ff5b4c000e/2d5c8383-b4dd-4e50-a76e-5d9de1ae531a/1491371a-c228-41d9-8946-b539dbebb3b9"
@@
           (reference "R17") (unit 1)
         )
+        (path "/99cd3e15-4eb6-4cbb-8726-789aedd3df15/c3b70d9b-0dcb-4344-9507-13ff5b4c000e/2d5c8383-b4dd-4e50-a76e-5d9de1ae531a/eab0e57f-22d7-4e2c-8f9b-b1863d6f54c5"
+          (reference "R2") (unit 1)
+        )
+        (path "/99cd3e15-4eb6-4cbb-8726-789aedd3df15/c3b70d9b-0dcb-4344-9507-13ff5b4c000e/2d5c8383-b4dd-4e50-a76e-5d9de1ae531a"
+          (reference "R35") (unit 1)
+        )
+        (path "/99cd3e15-4eb6-4cbb-8726-789aedd3df15/c3b70d9b-0dcb-4344-9507-13ff5b4c000e/3abb0ef0-3dd5-4818-a187-7e9bc43bafd4"
+          (reference "R8") (unit 1)
+        )
+        (path "/99cd3e15-4eb6-4cbb-8726-789aedd3df15/c3b70d9b-0dcb-4344-9507-13ff5b4c000e/2d5c8383-b4dd-4e50-a76e-5d9de1ae531a/6f15d501-5fa4-4bfe-a53d-adacae284de5"
+          (reference "R14") (unit 1)
+        )
       )

Commit message: WIP
Other:
- moved on the sheet: Q2, R19
Changed lines of the file:
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@@
 (kicad_sch (version 20230121) (generator eeschema)
   (paper "A5")
-  (junction (at 100.33 64.77) (diameter 0) (color 0 0 0 0)
+  (junction (at 106.68 68.58) (diameter 0) (color 0 0 0 0)
   )
-  (junction (at 115.57 54.61) (diameter 0) (color 0 0 0 0)
+  (junction (at 121.92 58.42) (diameter 0) (color 0 0 0 0)
   )
-  (junction (at 115.57 64.77) (diameter 0) (color 0 0 0 0)
+  (junction (at 121.92 68.58) (diameter 0) (color 0 0 0 0)
   )
-  (polyline (pts (xy 99.06 55.88) (xy 100.33 55.88))
+  (polyline (pts (xy 105.41 59.69) (xy 106.68 59.69))
     (stroke (width 0) (type default))
   )
-  (wire (pts (xy 115.57 52.07) (xy 115.57 54.61))
+  (wire (pts (xy 121.92 55.88) (xy 121.92 58.42))
     (stroke (width 0) (type default))
   )
-  (wire (pts (xy 100.33 64.77) (xy 102.87 64.77))
+  (wire (pts (xy 106.68 68.58) (xy 109.22 68.58))
     (stroke (width 0) (type default))
   )
-  (wire (pts (xy 107.95 57.15) (xy 107.95 54.61))
+  (wire (pts (xy 114.3 60.96) (xy 114.3 58.42))
     (stroke (width 0) (type default))
   )
-  (wire (pts (xy 115.57 64.77) (xy 127 64.77))
+  (wire (pts (xy 121.92 68.58) (xy 133.35 68.58))
     (stroke (width 0) (type default))
   )
-  (polyline (pts (xy 100.33 62.23) (xy 100.33 60.96))
+  (polyline (pts (xy 106.68 66.04) (xy 106.68 64.77))
     (stroke (width 0) (type default))
   )
-  (polyline (pts (xy 100.33 54.61) (xy 100.33 55.88))
+  (polyline (pts (xy 106.68 58.42) (xy 106.68 59.69))
     (stroke (width 0) (type default))
   )
-  (wire (pts (xy 100.33 62.23) (xy 100.33 64.77))
+  (wire (pts (xy 106.68 66.04) (xy 106.68 68.58))
     (stroke (width 0) (type default))
   )
-  (wire (pts (xy 88.9 64.77) (xy 100.33 64.77))
+  (wire (pts (xy 95.25 68.58) (xy 106.68 68.58))
     (stroke (width 0) (type default))
   )
-  (wire (pts (xy 115.57 54.61) (xy 115.57 64.77))
+  (wire (pts (xy 121.92 58.42) (xy 121.92 68.58))
     (stroke (width 0) (type default))
   )
-  (polyline (pts (xy 100.33 55.88) (xy 101.6 55.88))
+  (polyline (pts (xy 106.68 59.69) (xy 107.95 59.69))
     (stroke (width 0) (type default))
   )
-  (wire (pts (xy 113.03 64.77) (xy 115.57 64.77))
+  (wire (pts (xy 119.38 68.58) (xy 121.92 68.58))
     (stroke (width 0) (type default))
   )
-  (polyline (pts (xy 101.6 55.88) (xy 101.6 60.96))
+  (polyline (pts (xy 107.95 59.69) (xy 107.95 64.77))
     (stroke (width 0) (type default))
   )
-  (polyline (pts (xy 100.33 60.96) (xy 99.06 60.96))
+  (polyline (pts (xy 106.68 64.77) (xy 105.41 64.77))
     (stroke (width 0) (type default))
   )
-  (wire (pts (xy 107.95 54.61) (xy 115.57 54.61))
+  (wire (pts (xy 114.3 58.42) (xy 121.92 58.42))
     (stroke (width 0) (type default))
   )
-  (polyline (pts (xy 99.06 60.96) (xy 99.06 55.88))
+  (polyline (pts (xy 105.41 64.77) (xy 105.41 59.69))
     (stroke (width 0) (type default))
   )
-  (polyline (pts (xy 100.33 60.96) (xy 101.6 60.96))
+  (polyline (pts (xy 106.68 64.77) (xy 107.95 64.77))
     (stroke (width 0) (type default))
   )
@@
   )
   (text "Pro obousměrnou komunikaci \nje použit externí pull-up rezistor"
-    (at 64.77 60.96 0)
+    (at 71.12 64.77 0)
     (effects (font (size 1.27 1.27)) (justify left bottom))
   )
-  (text "HV-VCC" (at 96.52 53.34 0)
+  (text "HV-VCC" (at 102.87 57.15 0)
     (effects (font (size 1.27 1.27)) (justify left bottom))
   )
-  (hierarchical_label "LVD" (shape output) (at 127 64.77 0) (fields_autoplaced)
+  (hierarchical_label "LVD" (shape output) (at 133.35 68.58 0) (fields_autoplaced)
     (effects (font (size 1.27 1.27)) (justify left))
   )
-  (hierarchical_label "LV-VCC" (shape output) (at 115.57 44.45 90) (fields_autoplaced)
+  (hierarchical_label "LV-VCC" (shape output) (at 121.92 48.26 90) (fields_autoplaced)
     (effects (font (size 1.27 1.27)) (justify left))
   )
-  (hierarchical_label "HVD" (shape input) (at 88.9 64.77 180) (fields_autoplaced)
+  (hierarchical_label "HVD" (shape input) (at 95.25 68.58 180) (fields_autoplaced)
     (effects (font (size 1.27 1.27)) (justify right))
   )
-  (symbol (lib_id "Device:Q_NMOS_DGS") (at 107.95 62.23 90) (mirror x) (unit 1)
+  (symbol (lib_id "Device:Q_NMOS_DGS") (at 114.3 66.04 90) (mirror x) (unit 1)
     (in_bom yes) (on_board yes) (dnp no)
-    (property "Reference" "Q2" (at 109.22 71.12 90)
+    (property "Reference" "Q2" (at 115.57 74.93 90)
       (effects (font (size 1.27 1.27)) (justify left))
     )
-    (property "Value" "Q_NMOS_DGS" (at 114.3 68.58 90)
+    (property "Value" "Q_NMOS_DGS" (at 120.65 72.39 90)
       (effects (font (size 1.27 1.27)) (justify left))
     )
-    (property "Footprint" "Package_TO_SOT_SMD:SOT-723" (at 105.41 67.31 0)
+    (property "Footprint" "Package_TO_SOT_SMD:SOT-723" (at 111.76 71.12 0)
       (effects (font (size 1.27 1.27)) hide)
     )
-    (property "Datasheet" "https://datasheet.lcsc.com/lcsc/2201121900_ROHM-Semicon-RYM002N05GT2CL_C2941617.pdf" (at 107.95 62.23 0)
+    (property "Datasheet" "https://datasheet.lcsc.com/lcsc/2201121900_ROHM-Semicon-RYM002N05GT2CL_C2941617.pdf" (at 114.3 66.04 0)
       (effects (font (size 1.27 1.27)) hide)
     )
-    (property "LCSC" "C2941617" (at 107.95 62.23 0)
+    (property "LCSC" "C2941617" (at 114.3 66.04 0)
       (effects (font (size 1.27 1.27)) hide)
     )
-    (property "Basic/Extended" "E" (at 107.95 62.23 0)
+    (property "Basic/Extended" "E" (at 114.3 66.04 0)
       (effects (font (size 1.27 1.27)) hide)
     )
-    (property "JLCPCB_CORRECTION" "" (at 107.95 62.23 0)
+    (property "JLCPCB_CORRECTION" "" (at 114.3 66.04 0)
       (effects (font (size 1.27 1.27)) hide)
     )
@@
     )
   )
-  (symbol (lib_id "Device:R") (at 115.57 48.26 0) (unit 1)
+  (symbol (lib_id "Device:R") (at 121.92 52.07 0) (unit 1)
     (in_bom yes) (on_board yes) (dnp no)
-    (property "Reference" "R19" (at 118.11 46.99 0)
+    (property "Reference" "R19" (at 124.46 50.8 0)
       (effects (font (size 1.27 1.27)) (justify left))
     )
-    (property "Value" "10k" (at 118.11 49.53 0)
+    (property "Value" "10k" (at 124.46 53.34 0)
       (effects (font (size 1.27 1.27)) (justify left))
     )
-    (property "Footprint" "Resistor_SMD:R_0402_1005Metric" (at 113.792 48.26 90)
+    (property "Footprint" "Resistor_SMD:R_0402_1005Metric" (at 120.142 52.07 90)
       (effects (font (size 1.27 1.27)) hide)
     )
-    (property "Datasheet" "~" (at 115.57 48.26 0)
+    (property "Datasheet" "~" (at 121.92 52.07 0)
       (effects (font (size 1.27 1.27)) hide)
     )
-    (property "LCSC" "C25744" (at 115.57 48.26 0)
+    (property "LCSC" "C25744" (at 121.92 52.07 0)
       (effects (font (size 1.27 1.27)) hide)
     )
-    (property "JLCPCB_CORRECTION" "0;0;0" (at 115.57 48.26 0)
+    (property "JLCPCB_CORRECTION" "0;0;0" (at 121.92 52.07 0)
       (effects (font (size 1.27 1.27)) hide)
     )

Commit message: Zavazbení zapínání
Parts:
- Q2: footprint Package_TO_SOT_SMD:SOT-723 -> Package_TO_SOT_SMD:SOT-23; LCSC C2941617 -> C10487
Changed lines of the file:
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@@
       (effects (font (size 1.27 1.27)) (justify left))
     )
-    (property "Footprint" "Package_TO_SOT_SMD:SOT-723" (at 111.76 71.12 0)
+    (property "Footprint" "Package_TO_SOT_SMD:SOT-23" (at 111.76 71.12 0)
       (effects (font (size 1.27 1.27)) hide)
     )
-    (property "Datasheet" "https://datasheet.lcsc.com/lcsc/2201121900_ROHM-Semicon-RYM002N05GT2CL_C2941617.pdf" (at 114.3 66.04 0)
+    (property "Datasheet" "https://datasheet.lcsc.com/lcsc/1808272021_Vishay-Intertech-SI2301CDS-T1-GE3_C10487.pdf" (at 114.3 66.04 0)
       (effects (font (size 1.27 1.27)) hide)
     )
-    (property "LCSC" "C2941617" (at 114.3 66.04 0)
+    (property "LCSC" "C10487" (at 114.3 66.04 0)
       (effects (font (size 1.27 1.27)) hide)
     )
