File: hw/ZakladniElektronika/HlavniDeska/Zdroj.kicad_sch (KiCad schematic)
At the start: 28 parts, among them Q10 Q_PMOS_DGS-L, SW1 ON, U17 BateriCell_2x, U7 SL8261D-G3JE

Commit message: WIP
Parts:
- Q? (x3): symbol Device:Q_NMOS_DGS -> RKL-Uncategorized:Si7112DN
Connections:
- net GND: now also Q?.1 (S), Q?.2 (S)
- net VCC: now also Q?.4 (G); no longer Q?.2 (G)
- net at Q?.1 (S): now also C18.2, Q?.1 (S), Q?.2 (S), Q?.2 (S), Q?.3 (S), Q?.3 (S), R13.1, U7.6 (GND); no longer Q?.1 (D)
- net at U7.1 (OD): now also Q?.4 (G); no longer Q?.2 (G)
- net at U17.2 (-), U17.4 (-): now also Q?.5 (D); no longer Q?.1 (D)
- net at U7.3 (OC): now also Q?.4 (G); no longer Q?.2 (G)
- new net: Q?.5 (D), Q?.5 (D)
Other:
- moved on the sheet: Q?
Changed lines of the file:
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@@
+    (stroke (width 0) (type default))
+  )
+  (wire (pts (xy 109.22 50.8) (xy 109.22 81.28))
     (stroke (width 0) (type default))
   )
@@
     (stroke (width 0) (type default))
   )
+  (wire (pts (xy 88.9 121.92) (xy 86.36 121.92))
+    (stroke (width 0) (type default))
+  )
   (wire (pts (xy 208.28 76.2) (xy 208.28 81.28))
     (stroke (width 0) (type default))
   )
-  (wire (pts (xy 88.9 121.92) (xy 86.36 121.92))
-    (stroke (width 0) (type default))
-  )
   (wire (pts (xy 160.02 50.8) (xy 215.9 50.8))
     (stroke (width 0) (type default))
@@
   )
   (wire (pts (xy 179.07 82.55) (xy 179.07 88.9))
-    (stroke (width 0) (type default))
-  )
-  (wire (pts (xy 109.22 81.28) (xy 109.22 50.8))
     (stroke (width 0) (type default))
   )
@@
   (symbol (lib_id "Switch:SW_Push") (at 127 129.54 90) (unit 1)
     (in_bom yes) (on_board yes) (dnp no)
-    (property "Reference" "SW1" (at 114.3 128.27 90)
+    (property "Reference" "SW1" (at 119.38 128.27 90)
       (effects (font (size 1.27 1.27)) (justify right))
     )
-    (property "Value" "ON" (at 114.3 130.81 90)
+    (property "Value" "ON" (at 119.38 130.81 90)
       (effects (font (size 1.27 1.27)) (justify right))
     )
@@
     )
   )
-  (symbol (lib_id "Device:Q_NMOS_DGS") (at 190.5 86.36 270) (unit 1)
-    (in_bom yes) (on_board yes) (dnp no)
-    (property "Reference" "Q?" (at 190.5 92.71 90)
-      (effects (font (size 1.27 1.27)))
-    )
-    (property "Value" "Q_NMOS_DGS-P" (at 190.5 95.25 90)
-      (effects (font (size 1.27 1.27)))
-    )
-    (property "Footprint" "Package_SON:Diodes_PowerDI3333-8" (at 193.04 91.44 0)
-      (effects (font (size 1.27 1.27)) hide)
-    )
-    (property "Datasheet" "https://datasheet.lcsc.com/lcsc/2112021830_Vishay-Intertech-SI7112DN-T1-GE3_C2926777.pdf" (at 190.5 86.36 0)
-      (effects (font (size 1.27 1.27)) hide)
-    )
-    (property "LCSC" "C2926777" (at 190.5 86.36 0)
-      (effects (font (size 1.27 1.27)) hide)
-    )
-    (property "Basic/Extended" "E" (at 190.5 86.36 0)
-      (effects (font (size 1.27 1.27)) hide)
-    )
-    (property "JLCPCB_CORRECTION" "" (at 190.5 86.36 0)
+  (symbol (lib_name "Si7112DN_1") (lib_id "RKL-Uncategorized:Si7112DN") (at 190.5 88.9 180) (unit 1)
+    (in_bom yes) (on_board yes) (dnp no)
+    (property "Reference" "Q?" (at 190.5 92.71 0)
+      (effects (font (size 1.27 1.27)))
+    )
+    (property "Value" "Q_NMOS_DGS-P" (at 190.5 95.25 0)
+      (effects (font (size 1.27 1.27)))
+    )
+    (property "Footprint" "Package_SON:Diodes_PowerDI3333-8" (at 190.5 97.79 0)
+      (effects (font (size 1.27 1.27)) hide)
+    )
+    (property "Datasheet" "https://datasheet.lcsc.com/lcsc/2112021830_Vishay-Intertech-SI7112DN-T1-GE3_C2926777.pdf" (at 190.5 101.6 0)
+      (effects (font (size 1.27 1.27)) hide)
+    )
+    (property "LCSC" "C2926777" (at 190.5 104.14 0)
+      (effects (font (size 1.27 1.27)) hide)
+    )
+    (property "Basic/Extended" "E" (at 190.5 106.68 0)
+      (effects (font (size 1.27 1.27)) hide)
+    )
+    (property "JLCPCB_CORRECTION" "" (at 190.5 88.9 0)
       (effects (font (size 1.27 1.27)) hide)
     )
@@
     (pin "2")
     (pin "3")
+    (pin "4")
+    (pin "5")
     (instances
       (project "PowerManager"
@@
     )
   )
-  (symbol (lib_id "Device:Q_NMOS_DGS") (at 109.22 86.36 90) (mirror x) (unit 1)
-    (in_bom yes) (on_board yes) (dnp no)
-    (property "Reference" "Q?" (at 116.84 86.36 90)
-      (effects (font (size 1.27 1.27)) (justify left))
-    )
-    (property "Value" "Q_NMOS_DGS-P" (at 127 83.82 90)
-      (effects (font (size 1.27 1.27)) (justify left))
-    )
-    (property "Footprint" "Package_SON:Diodes_PowerDI3333-8" (at 106.68 91.44 0)
-      (effects (font (size 1.27 1.27)) hide)
-    )
-    (property "Datasheet" "https://datasheet.lcsc.com/lcsc/2112021830_Vishay-Intertech-SI7112DN-T1-GE3_C2926777.pdf" (at 109.22 86.36 0)
-      (effects (font (size 1.27 1.27)) hide)
-    )
-    (property "LCSC" "C2926777" (at 109.22 86.36 0)
-      (effects (font (size 1.27 1.27)) hide)
-    )
-    (property "Basic/Extended" "E" (at 109.22 86.36 0)
-      (effects (font (size 1.27 1.27)) hide)
-    )
-    (property "JLCPCB_CORRECTION" "" (at 109.22 86.36 0)
+  (symbol (lib_id "RKL-Uncategorized:Si7112DN") (at 109.22 88.9 0) (mirror x) (unit 1)
+    (in_bom yes) (on_board yes) (dnp no)
+    (property "Reference" "Q?" (at 114.3 86.36 0)
+      (effects (font (size 1.27 1.27)) (justify left))
+    )
+    (property "Value" "Q_NMOS_DGS-P" (at 110.49 83.82 0)
+      (effects (font (size 1.27 1.27)) (justify left))
+    )
+    (property "Footprint" "Package_SON:Diodes_PowerDI3333-8" (at 109.22 97.79 0)
+      (effects (font (size 1.27 1.27)) hide)
+    )
+    (property "Datasheet" "https://datasheet.lcsc.com/lcsc/2112021830_Vishay-Intertech-SI7112DN-T1-GE3_C2926777.pdf" (at 109.22 101.6 0)
+      (effects (font (size 1.27 1.27)) hide)
+    )
+    (property "LCSC" "C2926777" (at 109.22 104.14 0)
+      (effects (font (size 1.27 1.27)) hide)
+    )
+    (property "Basic/Extended" "E" (at 109.22 106.68 0)
+      (effects (font (size 1.27 1.27)) hide)
+    )
+    (property "JLCPCB_CORRECTION" "" (at 109.22 88.9 0)
       (effects (font (size 1.27 1.27)) hide)
     )
@@
     (pin "2")
     (pin "3")
+    (pin "4")
+    (pin "5")
     (instances
       (project "PowerManager"
@@
     )
   )
-  (symbol (lib_id "Device:Q_NMOS_DGS") (at 208.28 86.36 90) (mirror x) (unit 1)
-    (in_bom yes) (on_board yes) (dnp no)
-    (property "Reference" "Q?" (at 208.28 92.71 90)
-      (effects (font (size 1.27 1.27)))
-    )
-    (property "Value" "Q_NMOS_DGS-P" (at 208.28 95.25 90)
-      (effects (font (size 1.27 1.27)))
-    )
-    (property "Footprint" "Package_SON:Diodes_PowerDI3333-8" (at 205.74 91.44 0)
-      (effects (font (size 1.27 1.27)) hide)
-    )
-    (property "Datasheet" "https://datasheet.lcsc.com/lcsc/2112021830_Vishay-Intertech-SI7112DN-T1-GE3_C2926777.pdf" (at 208.28 86.36 0)
-      (effects (font (size 1.27 1.27)) hide)
-    )
-    (property "LCSC" "C2926777" (at 208.28 86.36 0)
-      (effects (font (size 1.27 1.27)) hide)
-    )
-    (property "Basic/Extended" "E" (at 208.28 86.36 0)
-      (effects (font (size 1.27 1.27)) hide)
-    )
-    (property "JLCPCB_CORRECTION" "" (at 208.28 86.36 0)
+  (symbol (lib_name "Si7112DN_2") (lib_id "RKL-Uncategorized:Si7112DN") (at 208.28 88.9 0) (mirror x) (unit 1)
+    (in_bom yes) (on_board yes) (dnp no)
+    (property "Reference" "Q?" (at 208.28 92.71 0)
+      (effects (font (size 1.27 1.27)))
+    )
+    (property "Value" "Q_NMOS_DGS-P" (at 208.28 95.25 0)
+      (effects (font (size 1.27 1.27)))
+    )
+    (property "Footprint" "Package_SON:Diodes_PowerDI3333-8" (at 208.28 97.79 0)
+      (effects (font (size 1.27 1.27)) hide)
+    )
+    (property "Datasheet" "https://datasheet.lcsc.com/lcsc/2112021830_Vishay-Intertech-SI7112DN-T1-GE3_C2926777.pdf" (at 208.28 101.6 0)
+      (effects (font (size 1.27 1.27)) hide)
+    )
+    (property "LCSC" "C2926777" (at 208.28 104.14 0)
+      (effects (font (size 1.27 1.27)) hide)
+    )
+    (property "Basic/Extended" "E" (at 208.28 106.68 0)
+      (effects (font (size 1.27 1.27)) hide)
+    )
+    (property "JLCPCB_CORRECTION" "" (at 208.28 88.9 0)
       (effects (font (size 1.27 1.27)) hide)
     )
@@
     (pin "2")
     (pin "3")
+    (pin "4")
+    (pin "5")
     (instances
       (project "PowerManager"

Commit message: PCB
Connections:
- net VCC: no longer TP2.1
- net at C18.2, Q?.1 (S), Q?.1 (S)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: now also TP2.1
Other:
- moved on the sheet: TP2
Changed lines of the file:
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@@
     (stroke (width 0) (type default))
   )
-  (wire (pts (xy 109.22 48.26) (xy 109.22 50.8))
+  (wire (pts (xy 160.02 91.44) (xy 160.02 88.9))
     (stroke (width 0) (type default))
   )
@@
     )
   )
-  (symbol (lib_id "Connector:TestPoint") (at 109.22 48.26 0) (unit 1)
-    (in_bom yes) (on_board yes) (dnp no)
-    (property "Reference" "TP2" (at 106.68 40.64 0)
-      (effects (font (size 1.27 1.27)) (justify left))
-    )
-    (property "Value" "TestPoint-BAT" (at 106.68 43.18 0)
-      (effects (font (size 1.27 1.27)) (justify left))
-    )
-    (property "Footprint" "Connector_Pin:Pin_D0.9mm_L10.0mm_W2.4mm_FlatFork" (at 114.3 48.26 0)
-      (effects (font (size 1.27 1.27)) hide)
-    )
-    (property "Datasheet" "~" (at 114.3 48.26 0)
-      (effects (font (size 1.27 1.27)) hide)
-    )
-    (property "JLCPCB_IGNORE" "ignore" (at 109.22 48.26 0)
+  (symbol (lib_id "Connector:TestPoint") (at 160.02 91.44 180) (unit 1)
+    (in_bom yes) (on_board yes) (dnp no)
+    (property "Reference" "TP2" (at 160.02 99.06 0)
+      (effects (font (size 1.27 1.27)))
+    )
+    (property "Value" "TestPoint-BAT" (at 160.02 96.52 0)
+      (effects (font (size 1.27 1.27)))
+    )
+    (property "Footprint" "Connector_Pin:Pin_D0.9mm_L10.0mm_W2.4mm_FlatFork" (at 154.94 91.44 0)
+      (effects (font (size 1.27 1.27)) hide)
+    )
+    (property "Datasheet" "~" (at 154.94 91.44 0)
+      (effects (font (size 1.27 1.27)) hide)
+    )
+    (property "JLCPCB_IGNORE" "ignore" (at 160.02 91.44 0)
       (effects (font (size 1.27 1.27)) hide)
     )
@@
           (reference "C18") (unit 1)
         )
-        (path "/99cd3e15-4eb6-4cbb-8726-789aedd3df15/6a867e96-34ab-4d6c-a824-47bb4ec04e8c/347f0ed9-f7fd-4b78-93c0-d59ffe3f4044"
-          (reference "C78") (unit 1)
-        )
-        (path "/99cd3e15-4eb6-4cbb-8726-789aedd3df15/c3b70d9b-0dcb-4344-9507-13ff5b4c000e/aae02708-da26-44dd-a602-660fbe003309/fb40dfe9-3eea-4dc3-8528-de588088c9ea"
+        (path "/99cd3e15-4eb6-4cbb-8726-789aedd3df15/c3b70d9b-0dcb-4344-9507-13ff5b4c000e/aae02708-da26-44dd-a602-660fbe003309/fb40dfe9-3eea-4dc3-8528-de588088c9ea"
