File: hw/ZakladniElektronika/HlavniDeska/GPSKomunikacniModul.kicad_sch (KiCad schematic)
At the start: 15 parts, among them J3 Conn_2Rows-75Pins, U2 TXB0304RUT, U6 TXB0304RUT, U8 PCA9306DC

Commit message: WIP
Connections:
- no-connect marks 39 -> 31
Changed lines of the file:
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@@
   (no_connect (at 175.26 58.42))
   (no_connect (at 175.26 88.9))
-  (no_connect (at 175.26 101.6))
   (no_connect (at 161.29 116.84))
   (no_connect (at 161.29 91.44))
   (no_connect (at 161.29 66.04))
-  (no_connect (at 162.56 106.68))
   (no_connect (at 238.76 50.8))
   (no_connect (at 161.29 96.52))
   (no_connect (at 175.26 63.5))
   (no_connect (at 175.26 86.36))
-  (no_connect (at 175.26 104.14))
   (no_connect (at 161.29 93.98))
   (no_connect (at 175.26 81.28))
@@
   (no_connect (at 176.53 45.72))
   (no_connect (at 175.26 73.66))
-  (no_connect (at 175.26 109.22))
   (no_connect (at 161.29 101.6))
   (no_connect (at 175.26 66.04))
   (no_connect (at 175.26 71.12))
-  (no_connect (at 162.56 104.14))
-  (no_connect (at 175.26 106.68))
-  (no_connect (at 162.56 111.76))
   (no_connect (at 176.53 48.26))
   (no_connect (at 176.53 50.8))
   (no_connect (at 162.56 154.94))
   (no_connect (at 161.29 68.58))
-  (no_connect (at 162.56 109.22))
   (no_connect (at 161.29 99.06))
   (bus_entry (at 50.8 106.68) (size 2.54 -2.54)
@@
       (effects (font (size 1.27 1.27)) hide)
     )
-    (property "Datasheet" "~" (at 170.18 78.74 0)
+    (property "Datasheet" "https://datasheet.lcsc.com/lcsc/2010161204_LOTES-APCI0161-P001A_C841663.pdf" (at 170.18 78.74 0)
       (effects (font (size 1.27 1.27)) hide)
     )
@@
     (pin "10")
     (pin "11")
-    (pin "12")
-    (pin "13")
-    (pin "14")
-    (pin "15")
-    (pin "16")
-    (pin "17")
-    (pin "18")
-    (pin "19")
     (pin "2")
     (pin "20")

Commit message: PCB
Parts:
- removed R8: 10k, Resistor_SMD:R_0402_1005Metric, symbol Device:R
Changed lines of the file:
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@@
 (kicad_sch (version 20230121) (generator eeschema)
   (paper "A4")
-  (junction (at 194.31 96.52) (diameter 0) (color 0 0 0 0)
-  )
   (junction (at 177.8 68.58) (diameter 0) (color 0 0 0 1)
   )
@@
     (stroke (width 0) (type default))
   )
-  (wire (pts (xy 194.31 93.98) (xy 194.31 96.52))
-    (stroke (width 0) (type default))
-  )
   (wire (pts (xy 162.56 68.58) (xy 161.29 68.58))
     (stroke (width 0) (type default))
@@
     (stroke (width 0) (type default))
   )
-  (wire (pts (xy 194.31 96.52) (xy 218.44 96.52))
-    (stroke (width 0) (type default))
-  )
   (wire (pts (xy 160.02 25.4) (xy 160.02 33.02))
     (stroke (width 0) (type default) (color 255 26 33 1))
@@
     (stroke (width 0) (type default))
   )
-  (wire (pts (xy 175.26 96.52) (xy 194.31 96.52))
+  (wire (pts (xy 175.26 96.52) (xy 218.44 96.52))
     (stroke (width 0) (type default))
   )
@@
     (effects (font (size 1.27 1.27)) (justify left bottom))
   )
-  (label "INT" (at 195.58 96.52 0) (fields_autoplaced)
+  (label "INT" (at 180.34 96.52 0) (fields_autoplaced)
     (effects (font (size 1.27 1.27)) (justify left bottom))
   )
@@
   (hierarchical_label "FUL_CARD_POWER_OFF" (shape input) (at 46.99 119.38 180) (fields_autoplaced)
     (effects (font (size 1.27 1.27)) (justify right))
-  )
-  (hierarchical_label "3V3" (shape input) (at 194.31 86.36 90) (fields_autoplaced)
-    (effects (font (size 1.27 1.27)) (justify left))
   )
   (hierarchical_label "1V8" (shape input) (at 92.71 25.4 90) (fields_autoplaced)
@@
         )
       )
-    )
-  )
-  (symbol (lib_id "Device:R") (at 194.31 90.17 0) (unit 1)
-    (in_bom yes) (on_board yes) (dnp no)
-    (property "Reference" "R8" (at 196.85 88.9 0)
-      (effects (font (size 1.27 1.27)) (justify left))
-    )
-    (property "Value" "10k" (at 196.85 91.44 0)
-      (effects (font (size 1.27 1.27)) (justify left))
-    )
-    (property "Footprint" "Resistor_SMD:R_0402_1005Metric" (at 192.532 90.17 90)
-      (effects (font (size 1.27 1.27)) hide)
-    )
-    (property "Datasheet" "~" (at 194.31 90.17 0)
-      (effects (font (size 1.27 1.27)) hide)
-    )
-    (property "LCSC" "C25744" (at 194.31 90.17 0)
-      (effects (font (size 1.27 1.27)) hide)
-    )
-    (property "JLCPCB_CORRECTION" "0;0;0" (at 194.31 90.17 0)
-      (effects (font (size 1.27 1.27)) hide)
-    )
-    (property "Basic/Extended" "B" (at 194.31 90.17 0)
-      (effects (font (size 1.27 1.27)) hide)
-    )
-    (pin "1")
-    (pin "2")
-    (instances
-      (project "ZakladniElektronika"
-        (path "/99cd3e15-4eb6-4cbb-8726-789aedd3df15/c3b70d9b-0dcb-4344-9507-13ff5b4c000e/3abb0ef0-3dd5-4818-a187-7e9bc43bafd4"
-          (reference "R8") (unit 1)
-        )
-        (path "/99cd3e15-4eb6-4cbb-8726-789aedd3df15/c3b70d9b-0dcb-4344-9507-13ff5b4c000e/2d5c8383-b4dd-4e50-a76e-5d9de1ae531a"
-          (reference "R34") (unit 1)
-        )
-      )
-      (project "RB3203"
-        (path "/dc7f8a41-3453-4df6-94dc-e94521e89591/9c917b4f-c6c7-4191-9aaa-f982c264da50/e24a5136-2be4-44de-8181-85cee94a1626"
-          (reference "R?") (unit 1)
-        )
-      )

Commit message: AHS-V1
Parts:
- J3: JLCPCB_CORRECTION (none) -> 0;-2;0
- U2, U6: JLCPCB_CORRECTION (none) -> 0;0;-90
- U53: JLCPCB_CORRECTION (none) -> 0;2;0
- U8: JLCPCB_CORRECTION (none) -> 0;0;180
Changed lines of the file:
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@@
+      (effects (font (size 1.27 1.27)) hide)
+    )
+    (property "JLCPCB_CORRECTION" "0;2;0" (at 175.26 143.51 0)
       (effects (font (size 1.27 1.27)) hide)
     )
@@
     )
     (property "Basic/Extended" "E" (at 228.6 30.48 0)
+      (effects (font (size 1.27 1.27)) hide)
+    )
+    (property "JLCPCB_CORRECTION" "0;0;-90" (at 228.6 30.48 0)
       (effects (font (size 1.27 1.27)) hide)
     )
@@
       (effects (font (size 1.27 1.27)) hide)
     )
+    (property "JLCPCB_CORRECTION" "0;0;180" (at 80.01 91.44 0)
+      (effects (font (size 1.27 1.27)) hide)
+    )
     (pin "1")
     (pin "2")
@@
     )
     (property "Basic/Extended" "E" (at 170.18 78.74 0)
+      (effects (font (size 1.27 1.27)) hide)
+    )
+    (property "JLCPCB_CORRECTION" "0;-2;0" (at 170.18 78.74 0)
       (effects (font (size 1.27 1.27)) hide)
     )
@@
       (effects (font (size 1.27 1.27)) hide)
     )
+    (property "JLCPCB_CORRECTION" "0;0;-90" (at 80.01 38.1 0)
+      (effects (font (size 1.27 1.27)) hide)
+    )
