File: hw/ZakladniElektronika/HlavniDeska/GPSKomunikacniModul.kicad_sch (KiCad schematic)
At the start: 14 parts, among them J3 Conn_2Rows-75Pins, U2 TXB0304RUT, U6 TXB0304RUT, U8 PCA9306DC

Commit message: KiCad V8
Parts:
- renumbered D125 to LED6, R13 to R2, R5 to R24, R5 to R25, R5 to R31
