File: hw/ZakladniElektronika/HlavniDeska/NapajeciRozcesti.kicad_sch (KiCad schematic)
At the start: 32 parts, among them Q1 Q_PMOS_DGS, Q2 Q_PMOS_DGS, U11 150k, U12 100k, U13 TPS61088RHLR, U14 100k, U15 2N7002, U16 LD39200, U17 33n, U18 150k, U19 22u, U20 4.7u, U21 10uf, U22 22u, U23 100k, U24 2N7002, U25 3.92k, U26 10n, U27 2.2u, U28 22u, U29 100p, U3 22u, U30 56k, U31 17.4k, U32 150k, U5 10uf, U6 100n, U7 1.2u, U8 4.7u, U9 100n

Commit message: WIP
Parts:
- removed D122: D_Dual_CommonCathode_AAK_Parallel, Package_TO_SOT_SMD:SOT-723, symbol Device:D_Dual_CommonCathode_AAK_Parallel
- removed Q1, Q2: Q_PMOS_DGS, RBCX:JMSL0302AU, symbol Device:Q_PMOS_DGS
- removed U12, U14, U23: 100k, Resistor_SMD:R_0402_1005Metric, symbol B.B-rescue:R-Device-B.B-rescue-B.B-rescue
- removed U15, U24: 2N7002, Package_TO_SOT_SMD:SOT-23, symbol B.B-rescue:2N7002-Transistor_FET-B.B-rescue-B.B-rescue
- added C138 (x2): 1u, Resistor_SMD:R_0402_1005Metric, symbol Device:C
- added U5: 150k, Resistor_SMD:R_0402_1005Metric, symbol B.B-rescue:R-Device-B.B-rescue-B.B-rescue
- added U52: MCP1700x-180xxTT, Package_TO_SOT_SMD:SOT-23, symbol Regulator_Linear:MCP1700x-180xxTT
- C142: Basic/Extended (none) -> E; LCSC C52923 -> C1518208; info (none) -> 50V, X7R
- C150: renamed from U8; symbol B.B-rescue:C-Device-B.B-rescue-B.B-rescue -> Device:C
- C151: renamed from U9; symbol B.B-rescue:C-Device-B.B-rescue-B.B-rescue -> Device:C; Basic/Extended (none) -> B; LCSC C1525 -> C307331; info (none) -> 50V, X7R
- C152: renamed from U17; symbol B.B-rescue:C-Device-B.B-rescue-B.B-rescue -> Device:C
- C153: renamed from U19; symbol B.B-rescue:C-Device-B.B-rescue-B.B-rescue -> Device:C
- C154: renamed from U20; symbol B.B-rescue:C-Device-B.B-rescue-B.B-rescue -> Device:C
- C155: renamed from U21; symbol B.B-rescue:C-Device-B.B-rescue-B.B-rescue -> Device:C
- C156: renamed from U22; symbol B.B-rescue:C-Device-B.B-rescue-B.B-rescue -> Device:C
- C157: renamed from U26; symbol B.B-rescue:C-Device-B.B-rescue-B.B-rescue -> Device:C
- C158: renamed from U27; symbol B.B-rescue:C-Device-B.B-rescue-B.B-rescue -> Device:C
- C159: renamed from U28; symbol B.B-rescue:C-Device-B.B-rescue-B.B-rescue -> Device:C
- C160: renamed from U29; symbol B.B-rescue:C-Device-B.B-rescue-B.B-rescue -> Device:C
- C5: renamed from U3; symbol B.B-rescue:C-Device-B.B-rescue-B.B-rescue -> Device:C
- C6: renamed from U5; symbol B.B-rescue:C-Device-B.B-rescue-B.B-rescue -> Device:C
- C7: renamed from U6; symbol B.B-rescue:C-Device-B.B-rescue-B.B-rescue -> Device:C; Basic/Extended (none) -> B; LCSC C1525 -> C307331; info (none) -> 50V, X7R
- renumbered U7 to L6, U32 to R41, U18 to R44, U30 to R46, U31 to R47
Connections:
- net 3V3: now also C138.1, U52.3 (VI)
- net GND: now also R41.1, C138.2, C138.2, U52.1 (GND); no longer R41.2
- net VCC: now also U5.1
- net EN-5V: now reaches U13.2 (EN)
- net EN-5V: now also R41.2; no longer R41.1
- net at U16.5 (EN): now also U5.2
- new net 1V8: C138.1, U52.2 (VO)
Other:
- note added: "1V8 LDO"
- note added: "3V3 LDO"
- note added: "5V Step-UP:"
- note removed: "LDO"
- note removed: "Step-UP:"
- moved on the sheet: C142, C150, C151, C152, C153, C154, C155, C156, C157, C158, C159, C160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

Commit message: Zavazbení zapínání
Parts:
- renumbered U25 to R42, U11 to R43, U5 to R50
Changed lines of the file:
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@@
   (symbol (lib_id "B.B-rescue:R-Device-B.B-rescue-B.B-rescue") (at 162.56 129.54 0) (unit 1)
     (in_bom yes) (on_board yes) (dnp no)
-    (property "Reference" "U25" (at 164.338 128.3716 0)
+    (property "Reference" "R42" (at 164.338 128.3716 0)
       (effects (font (size 1.27 1.27)) (justify left))
     )
@@
       (project "ZakladniElektronika"
         (path "/99cd3e15-4eb6-4cbb-8726-789aedd3df15/c3b70d9b-0dcb-4344-9507-13ff5b4c000e/aae02708-da26-44dd-a602-660fbe003309/3940fef8-969a-4db4-8b0b-434b96d98566"
-          (reference "U25") (unit 1)
+          (reference "R42") (unit 1)
         )
       )
@@
   (symbol (lib_id "B.B-rescue:R-Device-B.B-rescue-B.B-rescue") (at 97.79 107.95 90) (unit 1)
     (in_bom yes) (on_board yes) (dnp no)
-    (property "Reference" "U11" (at 93.98 109.22 90)
+    (property "Reference" "R43" (at 93.98 109.22 90)
       (effects (font (size 1.27 1.27)) (justify left))
     )
@@
       (project "ZakladniElektronika"
         (path "/99cd3e15-4eb6-4cbb-8726-789aedd3df15/c3b70d9b-0dcb-4344-9507-13ff5b4c000e/aae02708-da26-44dd-a602-660fbe003309/3940fef8-969a-4db4-8b0b-434b96d98566"
-          (reference "U11") (unit 1)
+          (reference "R43") (unit 1)
         )
       )
@@
   (symbol (lib_id "B.B-rescue:R-Device-B.B-rescue-B.B-rescue") (at 91.44 64.77 90) (unit 1)
     (in_bom yes) (on_board yes) (dnp no)
-    (property "Reference" "U5" (at 87.63 66.04 90)
+    (property "Reference" "R50" (at 87.63 66.04 90)
       (effects (font (size 1.27 1.27)) (justify left))
     )
@@
       (project "ZakladniElektronika"
         (path "/99cd3e15-4eb6-4cbb-8726-789aedd3df15/c3b70d9b-0dcb-4344-9507-13ff5b4c000e/aae02708-da26-44dd-a602-660fbe003309/3940fef8-969a-4db4-8b0b-434b96d98566"
-          (reference "U5") (unit 1)
-        )
-      )
+          (reference "R50") (unit 1)
+        )
+      )

Commit message: USB_multiplexer a přehlednost
Other:
- moved on the sheet: R41
Changed lines of the file:
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@@
   (junction (at 162.56 123.19) (diameter 0) (color 0 0 0 0)
   )
+  (junction (at 95.25 123.19) (diameter 0) (color 0 0 0 0)
+  )
   (junction (at 88.9 97.79) (diameter 0) (color 0 0 0 0)
   )
@@
   )
   (junction (at 50.8 97.79) (diameter 0) (color 0 0 0 0)
-  )
-  (junction (at 96.52 123.19) (diameter 0) (color 0 0 0 0)
   )
   (no_connect (at 120.65 64.77))
@@
     (stroke (width 0) (type default))
   )
-  (wire (pts (xy 93.98 123.19) (xy 96.52 123.19))
+  (wire (pts (xy 92.71 123.19) (xy 95.25 123.19))
     (stroke (width 0) (type default))
   )
@@
     (stroke (width 0) (type default))
   )
-  (wire (pts (xy 96.52 123.19) (xy 96.52 125.73))
+  (wire (pts (xy 95.25 123.19) (xy 95.25 125.73))
     (stroke (width 0) (type default))
   )
@@
     (stroke (width 0) (type default))
   )
-  (wire (pts (xy 96.52 123.19) (xy 101.6 123.19))
+  (wire (pts (xy 95.25 123.19) (xy 101.6 123.19))
     (stroke (width 0) (type default))
   )
@@
     (stroke (width 0) (type default))
   )
-  (wire (pts (xy 96.52 133.35) (xy 96.52 140.97))
+  (wire (pts (xy 95.25 133.35) (xy 95.25 140.97))
     (stroke (width 0) (type default))
   )
@@
     (effects (font (size 1.27 1.27)) (justify right))
   )
-  (hierarchical_label "GND" (shape output) (at 110.49 140.97 270) (fields_autoplaced)
-    (effects (font (size 1.27 1.27)) (justify right))
-  )
-  (hierarchical_label "GND" (shape output) (at 127 39.37 270) (fields_autoplaced)
-    (effects (font (size 1.27 1.27)) (justify right))
-  )
-  (hierarchical_label "GND" (shape output) (at 137.16 113.03 270) (fields_autoplaced)
+  (hierarchical_label "GND" (shape passive) (at 76.2 123.19 270) (fields_autoplaced)
     (effects (font (size 1.27 1.27)) (justify right))
   )
@@
     (effects (font (size 1.27 1.27)) (justify left))
   )
-  (hierarchical_label "GND" (shape output) (at 149.86 140.97 270) (fields_autoplaced)
-    (effects (font (size 1.27 1.27)) (justify right))
-  )
-  (hierarchical_label "GND" (shape output) (at 107.95 72.39 270) (fields_autoplaced)
-    (effects (font (size 1.27 1.27)) (justify right))
-  )
-  (hierarchical_label "GND" (shape output) (at 124.46 113.03 270) (fields_autoplaced)
-    (effects (font (size 1.27 1.27)) (justify right))
-  )
-  (hierarchical_label "GND" (shape output) (at 107.95 39.37 270) (fields_autoplaced)
-    (effects (font (size 1.27 1.27)) (justify right))
-  )
-  (hierarchical_label "GND" (shape output) (at 113.03 140.97 270) (fields_autoplaced)
-    (effects (font (size 1.27 1.27)) (justify right))
-  )
-  (hierarchical_label "GND" (shape output) (at 162.56 140.97 270) (fields_autoplaced)
-    (effects (font (size 1.27 1.27)) (justify right))
-  )
-  (hierarchical_label "GND" (shape output) (at 175.26 140.97 270) (fields_autoplaced)
-    (effects (font (size 1.27 1.27)) (justify right))
-  )
-  (hierarchical_label "GND" (shape output) (at 100.33 140.97 270) (fields_autoplaced)
-    (effects (font (size 1.27 1.27)) (justify right))
-  )
-  (hierarchical_label "GND" (shape output) (at 137.16 140.97 270) (fields_autoplaced)
-    (effects (font (size 1.27 1.27)) (justify right))
-  )
-  (hierarchical_label "GND" (shape output) (at 88.9 39.37 270) (fields_autoplaced)
-    (effects (font (size 1.27 1.27)) (justify right))
-  )
-  (hierarchical_label "GND" (shape output) (at 63.5 123.19 270) (fields_autoplaced)
-    (effects (font (size 1.27 1.27)) (justify right))
-  )
-  (hierarchical_label "GND" (shape output) (at 129.54 72.39 270) (fields_autoplaced)
+  (hierarchical_label "GND" (shape passive) (at 69.85 72.39 270) (fields_autoplaced)
+    (effects (font (size 1.27 1.27)) (justify right))
+  )
+  (hierarchical_label "GND" (shape passive) (at 137.16 113.03 270) (fields_autoplaced)
+    (effects (font (size 1.27 1.27)) (justify right))
+  )
+  (hierarchical_label "GND" (shape passive) (at 63.5 123.19 270) (fields_autoplaced)
+    (effects (font (size 1.27 1.27)) (justify right))
+  )
+  (hierarchical_label "GND" (shape passive) (at 162.56 113.03 270) (fields_autoplaced)
+    (effects (font (size 1.27 1.27)) (justify right))
+  )
+  (hierarchical_label "GND" (shape passive) (at 95.25 140.97 270) (fields_autoplaced)
+    (effects (font (size 1.27 1.27)) (justify right))
+  )
+  (hierarchical_label "GND" (shape passive) (at 107.95 72.39 270) (fields_autoplaced)
+    (effects (font (size 1.27 1.27)) (justify right))
+  )
+  (hierarchical_label "GND" (shape passive) (at 100.33 140.97 270) (fields_autoplaced)
+    (effects (font (size 1.27 1.27)) (justify right))
+  )
+  (hierarchical_label "GND" (shape passive) (at 129.54 72.39 270) (fields_autoplaced)
+    (effects (font (size 1.27 1.27)) (justify right))
+  )
+  (hierarchical_label "GND" (shape passive) (at 113.03 140.97 270) (fields_autoplaced)
+    (effects (font (size 1.27 1.27)) (justify right))
+  )
+  (hierarchical_label "GND" (shape passive) (at 175.26 140.97 270) (fields_autoplaced)
+    (effects (font (size 1.27 1.27)) (justify right))
+  )
+  (hierarchical_label "GND" (shape passive) (at 184.15 120.65 270) (fields_autoplaced)
+    (effects (font (size 1.27 1.27)) (justify right))
+  )
+  (hierarchical_label "GND" (shape passive) (at 107.95 39.37 270) (fields_autoplaced)
     (effects (font (size 1.27 1.27)) (justify right))
   )
@@
     (effects (font (size 1.27 1.27)) (justify left))
   )
-  (hierarchical_label "GND" (shape output) (at 96.52 140.97 270) (fields_autoplaced)
+  (hierarchical_label "GND" (shape passive) (at 162.56 140.97 270) (fields_autoplaced)
     (effects (font (size 1.27 1.27)) (justify right))
   )
@@
     (effects (font (size 1.27 1.27)) (justify left))
   )
-  (hierarchical_label "GND" (shape output) (at 184.15 120.65 270) (fields_autoplaced)
-    (effects (font (size 1.27 1.27)) (justify right))
-  )
-  (hierarchical_label "GND" (shape output) (at 162.56 113.03 270) (fields_autoplaced)
-    (effects (font (size 1.27 1.27)) (justify right))
-  )
-  (hierarchical_label "GND" (shape output) (at 140.97 72.39 270) (fields_autoplaced)
-    (effects (font (size 1.27 1.27)) (justify right))
-  )
-  (hierarchical_label "GND" (shape output) (at 124.46 140.97 270) (fields_autoplaced)
-    (effects (font (size 1.27 1.27)) (justify right))
-  )
-  (hierarchical_label "EN-5V" (shape input) (at 93.98 123.19 180) (fields_autoplaced)
-    (effects (font (size 1.27 1.27)) (justify right))
-  )
-  (hierarchical_label "GND" (shape output) (at 76.2 123.19 270) (fields_autoplaced)
-    (effects (font (size 1.27 1.27)) (justify right))
-  )
-  (hierarchical_label "GND" (shape output) (at 149.86 113.03 270) (fields_autoplaced)
-    (effects (font (size 1.27 1.27)) (justify right))
-  )
-  (hierarchical_label "GND" (shape output) (at 50.8 123.19 270) (fields_autoplaced)
-    (effects (font (size 1.27 1.27)) (justify right))
-  )
-  (hierarchical_label "GND" (shape output) (at 69.85 72.39 270) (fields_autoplaced)
+  (hierarchical_label "GND" (shape passive) (at 140.97 72.39 270) (fields_autoplaced)
+    (effects (font (size 1.27 1.27)) (justify right))
+  )
+  (hierarchical_label "GND" (shape passive) (at 127 39.37 270) (fields_autoplaced)
+    (effects (font (size 1.27 1.27)) (justify right))
+  )
+  (hierarchical_label "GND" (shape passive) (at 137.16 140.97 270) (fields_autoplaced)
+    (effects (font (size 1.27 1.27)) (justify right))
+  )
+  (hierarchical_label "GND" (shape passive) (at 88.9 39.37 270) (fields_autoplaced)
+    (effects (font (size 1.27 1.27)) (justify right))
+  )
+  (hierarchical_label "GND" (shape passive) (at 124.46 113.03 270) (fields_autoplaced)
+    (effects (font (size 1.27 1.27)) (justify right))
+  )
+  (hierarchical_label "EN-5V" (shape input) (at 92.71 123.19 180) (fields_autoplaced)
+    (effects (font (size 1.27 1.27)) (justify right))
+  )
+  (hierarchical_label "GND" (shape passive) (at 149.86 140.97 270) (fields_autoplaced)
+    (effects (font (size 1.27 1.27)) (justify right))
+  )
+  (hierarchical_label "GND" (shape passive) (at 124.46 140.97 270) (fields_autoplaced)
+    (effects (font (size 1.27 1.27)) (justify right))
+  )
+  (hierarchical_label "GND" (shape passive) (at 110.49 140.97 270) (fields_autoplaced)
+    (effects (font (size 1.27 1.27)) (justify right))
+  )
+  (hierarchical_label "GND" (shape passive) (at 50.8 123.19 270) (fields_autoplaced)
+    (effects (font (size 1.27 1.27)) (justify right))
+  )
+  (hierarchical_label "GND" (shape passive) (at 149.86 113.03 270) (fields_autoplaced)
     (effects (font (size 1.27 1.27)) (justify right))
   )
@@
     )
   )
-  (symbol (lib_id "B.B-rescue:R-Device-B.B-rescue-B.B-rescue") (at 96.52 129.54 180) (unit 1)
-    (in_bom yes) (on_board yes) (dnp no)
-    (property "Reference" "R41" (at 93.98 128.27 0)
-      (effects (font (size 1.27 1.27)) (justify left))
-    )
-    (property "Value" "150k" (at 93.98 130.81 0)
-      (effects (font (size 1.27 1.27)) (justify left))
-    )
-    (property "Footprint" "Resistor_SMD:R_0402_1005Metric" (at 98.298 129.54 90)
-      (effects (font (size 1.27 1.27)) hide)
-    )
-    (property "Datasheet" "~" (at 96.52 129.54 0)
-      (effects (font (size 1.27 1.27)) hide)
-    )
-    (property "LCSC" "C25755" (at 96.52 129.54 0)
-      (effects (font (size 1.27 1.27)) hide)
-    )
+  (symbol (lib_id "B.B-rescue:R-Device-B.B-rescue-B.B-rescue") (at 95.25 129.54 180) (unit 1)
+    (in_bom yes) (on_board yes) (dnp no)
+    (property "Reference" "R41" (at 92.71 128.27 0)
+      (effects (font (size 1.27 1.27)) (justify left))
+    )
+    (property "Value" "150k" (at 92.71 130.81 0)
+      (effects (font (size 1.27 1.27)) (justify left))
+    )
+    (property "Footprint" "Resistor_SMD:R_0402_1005Metric" (at 97.028 129.54 90)
+      (effects (font (size 1.27 1.27)) hide)
+    )
+    (property "Datasheet" "~" (at 95.25 129.54 0)
+      (effects (font (size 1.27 1.27)) hide)
+    )
+    (property "LCSC" "C25755" (at 95.25 129.54 0)
+      (effects (font (size 1.27 1.27)) hide)
+    )
