File: hw/ZakladniElektronika/HlavniDeska/NapajeciRozcesti.kicad_sch (KiCad schematic)
At the start: 26 parts, among them U11 NCP708, U3 TPS61088RHLR, U52 MCP1700x-180xxTT

Commit message: KiCad V8
Parts:
- renumbered C138 to C148, C138 to C149
