File: hw/ZakladniElektronika/HlavniDeska/Nabijecka.kicad_sch (KiCad schematic)
At the start: 17 parts, among them U5 10u, U9 BQ25895RTW

Commit message: KiCad V8
Parts:
- renumbered U5 to C145, U5 to C146, U5 to C147, C150 to C164, C3 to C166, D126 to LED5, R13 to R18, R13 to R19, R13 to R20, R17 to R21, R17 to R71, TP4 to TP6, TP4 to TP7
