File: hw/ZakladniElektronika/HlavniDeska/USB.kicad_sch (KiCad schematic)
At the start: 18 parts, among them J2 USB_C_Receptacle_USB2.0, U13 TPD4E02B04DQA, U4 AP33772

Commit message: PCB
Connections:
- net VUSB renamed VBUS
Changed lines of the file:
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@@
     (effects (font (size 1.27 1.27)) (justify right))
   )
-  (hierarchical_label "VUSB" (shape output) (at 233.68 67.31 0) (fields_autoplaced)
+  (hierarchical_label "VBUS" (shape output) (at 233.68 67.31 0) (fields_autoplaced)
     (effects (font (size 1.27 1.27)) (justify left))
   )
@@
   (symbol (lib_id "Device:C") (at 154.94 73.66 0) (unit 1)
     (in_bom yes) (on_board yes) (dnp no)
-    (property "Reference" "C136" (at 156.21 71.12 0)
-      (effects (font (size 1.27 1.27)) (justify left))
-    )
-    (property "Value" "10u" (at 156.21 76.2 0)
+    (property "Reference" "C136" (at 157.48 72.39 0)
+      (effects (font (size 1.27 1.27)) (justify left))
+    )
+    (property "Value" "10u" (at 157.48 74.93 0)
       (effects (font (size 1.27 1.27)) (justify left))
     )
@@
   (symbol (lib_id "Device:R") (at 227.33 105.41 270) (unit 1)
     (in_bom yes) (on_board yes) (dnp no)
-    (property "Reference" "R12" (at 228.6 102.87 90)
-      (effects (font (size 1.27 1.27)))
-    )
-    (property "Value" "10k" (at 224.79 102.87 90)
+    (property "Reference" "R12" (at 227.33 100.33 90)
+      (effects (font (size 1.27 1.27)))
+    )
+    (property "Value" "10k" (at 227.33 102.87 90)
       (effects (font (size 1.27 1.27)))
     )
@@
   (symbol (lib_id "Device:C") (at 186.69 81.28 90) (unit 1)
     (in_bom yes) (on_board yes) (dnp no)
-    (property "Reference" "C137" (at 185.42 74.93 90)
+    (property "Reference" "C137" (at 186.69 74.93 90)
       (effects (font (size 1.27 1.27)))
     )
@@
   (symbol (lib_id "Device:R") (at 167.64 81.28 180) (unit 1)
     (in_bom yes) (on_board yes) (dnp no)
-    (property "Reference" "R5" (at 165.1 82.55 90)
-      (effects (font (size 1.27 1.27)) (justify left))
-    )
-    (property "Value" "4.7k" (at 165.1 77.47 90)
-      (effects (font (size 1.27 1.27)) (justify left))
+    (property "Reference" "R5" (at 170.18 80.01 0)
+      (effects (font (size 1.27 1.27)) (justify right))
+    )
+    (property "Value" "4.7k" (at 170.18 82.55 0)
+      (effects (font (size 1.27 1.27)) (justify right))
     )
     (property "Footprint" "Resistor_SMD:R_0402_1005Metric" (at 169.418 81.28 90)
@@
   (symbol (lib_id "Device:C") (at 223.52 118.11 180) (unit 1)
     (in_bom yes) (on_board yes) (dnp no)
-    (property "Reference" "C140" (at 228.6 116.84 0)
-      (effects (font (size 1.27 1.27)))
-    )
-    (property "Value" "100n" (at 229.87 119.38 0)
-      (effects (font (size 1.27 1.27)))
+    (property "Reference" "C140" (at 226.06 116.84 0)
+      (effects (font (size 1.27 1.27)) (justify right))
+    )
+    (property "Value" "100n" (at 226.06 119.38 0)
+      (effects (font (size 1.27 1.27)) (justify right))
     )
     (property "Footprint" "Capacitor_SMD:C_0402_1005Metric" (at 222.5548 114.3 0)
@@
   (symbol (lib_id "Device:C") (at 193.04 118.11 180) (unit 1)
     (in_bom yes) (on_board yes) (dnp no)
-    (property "Reference" "C139" (at 198.12 116.84 0)
-      (effects (font (size 1.27 1.27)))
-    )
-    (property "Value" "100n" (at 199.39 119.38 0)
-      (effects (font (size 1.27 1.27)))
+    (property "Reference" "C139" (at 195.58 116.84 0)
+      (effects (font (size 1.27 1.27)) (justify right))
+    )
+    (property "Value" "100n" (at 195.58 119.38 0)
+      (effects (font (size 1.27 1.27)) (justify right))
     )
     (property "Footprint" "Capacitor_SMD:C_0402_1005Metric" (at 192.0748 114.3 0)
@@
   (symbol (lib_id "Device:R") (at 241.3 118.11 180) (unit 1)
     (in_bom yes) (on_board yes) (dnp no)
-    (property "Reference" "R13" (at 238.76 119.38 90)
-      (effects (font (size 1.27 1.27)) (justify left))
-    )
-    (property "Value" "4.7k" (at 238.76 114.3 90)
-      (effects (font (size 1.27 1.27)) (justify left))
+    (property "Reference" "R13" (at 243.84 116.84 0)
+      (effects (font (size 1.27 1.27)) (justify right))
+    )
+    (property "Value" "4.7k" (at 243.84 119.38 0)
+      (effects (font (size 1.27 1.27)) (justify right))
     )
     (property "Footprint" "Resistor_SMD:R_0402_1005Metric" (at 243.078 118.11 90)
@@
   (symbol (lib_id "Device:C") (at 182.88 118.11 0) (mirror y) (unit 1)
     (in_bom yes) (on_board yes) (dnp no)
-    (property "Reference" "C138" (at 190.5 116.84 0)
-      (effects (font (size 1.27 1.27)) (justify left))
-    )
-    (property "Value" "1u" (at 190.5 119.38 0)
-      (effects (font (size 1.27 1.27)) (justify left))
+    (property "Reference" "C138" (at 185.42 116.84 0)
+      (effects (font (size 1.27 1.27)) (justify right))
+    )
+    (property "Value" "1u" (at 185.42 119.38 0)
+      (effects (font (size 1.27 1.27)) (justify right))
     )
     (property "Footprint" "Capacitor_SMD:C_0402_1005Metric" (at 181.9148 121.92 0)

Commit message: AHS-V1
Parts:
- J2: JLCPCB_CORRECTION 0;-1;0 -> 0;-3.5;0
- U13: JLCPCB_CORRECTION (none) -> 0;0;-90
Changed lines of the file:
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@@
       (effects (font (size 1.27 1.27)) hide)
     )
-    (property "JLCPCB_CORRECTION" "0;-1;0" (at 71.12 58.42 0)
+    (property "JLCPCB_CORRECTION" "0;-3.5;0" (at 71.12 58.42 0)
       (effects (font (size 1.27 1.27)) hide)
     )
@@
       (effects (font (size 1.27 1.27)) hide)
     )
+    (property "JLCPCB_CORRECTION" "0;0;-90" (at 96.52 92.71 0)
+      (effects (font (size 1.27 1.27)) hide)
+    )

Commit message: Hw PCB
Parts:
- removed C136: 10u, Capacitor_SMD:C_0805_2012Metric, symbol Device:C
- removed C137, C139, C140: 100n, Capacitor_SMD:C_0402_1005Metric, symbol Device:C
- removed C138, C141: 1u, Capacitor_SMD:C_0402_1005Metric, symbol Device:C
- removed D123: PTVSHC3N24, RKL-StandardPackages:DFN3-2x2, symbol RKL-Uncategorized:PTVSHC3N24
- removed LED3, LED4: red, LED_SMD:LED_0603_1608Metric, symbol Device:LED
- removed R11: 10m, Resistor_SMD:R_1206_3216Metric, symbol Device:R
- removed R12: 10k, Resistor_SMD:R_0402_1005Metric, symbol Device:R
- removed R13, R5: 4.7k, Resistor_SMD:R_0402_1005Metric, symbol Device:R
- removed U4: AP33772, Package_DFN_QFN:QFN-24-1EP_4x4mm_P0.5mm_EP2.6x2.6mm, symbol RKL-BusCnverters:AP33772
Connections:
- net V_USB is gone; now on net VBUS: J2.A4 (VBUS), J2.A9 (VBUS), J2.B4 (VBUS), J2.B9 (VBUS)
- net D+: now also U13.4 (IO3); no longer U13.5 (IO4)
- net D-: now also U13.2 (IO2); no longer U13.4 (IO3)
- net USB_CC1: no longer U13.1 (IO1)
- net USB_CC2: no longer U13.2 (IO2)
- net VBUS: now also U13.1 (IO1), U13.5 (IO4)
- no-connect marks 15 -> 10
Other:
- note removed: "PD jednatel"
- moved on the sheet: J2, R3, R4, U13
