File: hw/ZakladniElektronika/HlavniDeska/ModuloviKonektor.kicad_sch (KiCad schematic)
At the start: 7 parts, among them J4 Conn_01x07, U5 TPD4E02B04DQA

Commit message: Hw PCB
Connections:
- net INT: now also U5.2 (IO2); no longer U5.4 (IO3)
- net USART-TX: now also U5.4 (IO3); no longer U5.2 (IO2)
Changed lines of the file:
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@@
 (kicad_sch
-	(version 20231120)
+	(version 20250114)
 	(generator "eeschema")
-	(generator_version "8.0")
+	(generator_version "9.0")
 	(paper "A5")
 	(junction
+		(at 91.44 58.42)
+		(diameter 0)
+		(color 0 0 0 0)
+	)
+	(junction
+		(at 86.36 66.04)
+		(diameter 0)
+		(color 0 0 0 0)
+	)
+	(junction
 		(at 83.82 50.8)
 		(diameter 0)
@@
 	)
 	(junction
-		(at 86.36 58.42)
-		(diameter 0)
-		(color 0 0 0 0)
-	)
-	(junction
 		(at 109.22 50.8)
 		(diameter 0)
@@
 	)
 	(junction
-		(at 91.44 66.04)
-		(diameter 0)
-		(color 0 0 0 0)
-	)
-	(junction
 		(at 127 60.96)
 		(diameter 0)
@@
 	(wire
 		(pts
+			(xy 86.36 66.04) (xy 93.98 66.04)
+		)
+		(stroke
+			(width 0)
+			(type default)
+		)
+	)
+	(wire
+		(pts
 			(xy 124.46 53.34) (xy 129.54 53.34)
 		)
@@
 	(wire
 		(pts
-			(xy 86.36 58.42) (xy 86.36 73.66)
-		)
-		(stroke
-			(width 0)
-			(type default)
-		)
-	)
-	(wire
-		(pts
-			(xy 78.74 66.04) (xy 91.44 66.04)
+			(xy 91.44 58.42) (xy 91.44 73.66)
+		)
+		(stroke
+			(width 0)
+			(type default)
+		)
+	)
+	(wire
+		(pts
+			(xy 78.74 66.04) (xy 86.36 66.04)
 		)
 		(stroke
@@
 	(wire
 		(pts
-			(xy 91.44 66.04) (xy 91.44 73.66)
-		)
-		(stroke
-			(width 0)
-			(type default)
-		)
-	)
-	(wire
-		(pts
-			(xy 78.74 58.42) (xy 86.36 58.42)
+			(xy 86.36 66.04) (xy 86.36 73.66)
+		)
+		(stroke
+			(width 0)
+			(type default)
+		)
+	)
+	(wire
+		(pts
+			(xy 78.74 58.42) (xy 91.44 58.42)
 		)
 		(stroke
@@
 	(wire
 		(pts
-			(xy 91.44 66.04) (xy 93.98 66.04)
+			(xy 91.44 58.42) (xy 93.98 58.42)
 		)
 		(stroke
@@
 		(pts
 			(xy 83.82 50.8) (xy 93.98 50.8)
-		)
-		(stroke
-			(width 0)
-			(type default)
-		)
-	)
-	(wire
-		(pts
-			(xy 86.36 58.42) (xy 93.98 58.42)
 		)
 		(stroke
@@
 		(shape input)
 		(at 124.46 35.56 90)
-		(fields_autoplaced yes)
 		(effects
 			(font
@@
 		(shape bidirectional)
 		(at 127 68.58 270)
-		(fields_autoplaced yes)
 		(effects
 			(font
@@
 		(shape bidirectional)
 		(at 88.9 86.36 270)
-		(fields_autoplaced yes)
 		(effects
 			(font
@@
 		(shape output)
 		(at 78.74 66.04 180)
-		(fields_autoplaced yes)
 		(effects
 			(font
@@
 		(shape output)
 		(at 78.74 50.8 180)
-		(fields_autoplaced yes)
 		(effects
 			(font
@@
 		(shape input)
 		(at 78.74 58.42 180)
-		(fields_autoplaced yes)
 		(effects
 			(font
@@
 		(shape input)
 		(at 109.22 36.83 90)
-		(fields_autoplaced yes)
 		(effects
 			(font
@@
 		(shape input)
 		(at 119.38 36.83 90)
-		(fields_autoplaced yes)
-		(effects
-			(font
+		(effects
+			(font

Commit message: Bordel Hw
Connections:
- net 5V: now also U5.4 (IO3); no longer U5.5 (IO4)
- net INT: now also U5.5 (IO4); no longer U5.2 (IO2)
- net USART-TX: now also U5.2 (IO2); no longer U5.4 (IO3)
Other:
- moved on the sheet: U5
Changed lines of the file:
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@@
 	(paper "A5")
 	(junction
-		(at 91.44 58.42)
+		(at 81.28 50.8)
 		(diameter 0)
 		(color 0 0 0 0)
 	)
 	(junction
-		(at 86.36 66.04)
+		(at 83.82 58.42)
 		(diameter 0)
 		(color 0 0 0 0)
 	)
 	(junction
-		(at 83.82 50.8)
+		(at 91.44 66.04)
 		(diameter 0)
 		(color 0 0 0 0)
@@
 	(wire
 		(pts
-			(xy 86.36 66.04) (xy 93.98 66.04)
-		)
-		(stroke
-			(width 0)
-			(type default)
-		)
-	)
-	(wire
-		(pts
 			(xy 124.46 53.34) (xy 129.54 53.34)
 		)
@@
 	(wire
 		(pts
-			(xy 91.44 58.42) (xy 91.44 73.66)
-		)
-		(stroke
-			(width 0)
-			(type default)
-		)
-	)
-	(wire
-		(pts
-			(xy 78.74 66.04) (xy 86.36 66.04)
+			(xy 83.82 58.42) (xy 83.82 73.66)
+		)
+		(stroke
+			(width 0)
+			(type default)
+		)
+	)
+	(wire
+		(pts
+			(xy 78.74 66.04) (xy 91.44 66.04)
 		)
 		(stroke
@@
 	(wire
 		(pts
-			(xy 83.82 50.8) (xy 83.82 73.66)
+			(xy 81.28 50.8) (xy 93.98 50.8)
+		)
+		(stroke
+			(width 0)
+			(type default)
+		)
+	)
+	(wire
+		(pts
+			(xy 81.28 50.8) (xy 81.28 73.66)
+		)
+		(stroke
+			(width 0)
+			(type default)
+		)
+	)
+	(wire
+		(pts
+			(xy 91.44 66.04) (xy 93.98 66.04)
+		)
+		(stroke
+			(width 0)
+			(type default)
+		)
+	)
+	(wire
+		(pts
+			(xy 83.82 58.42) (xy 93.98 58.42)
+		)
+		(stroke
+			(width 0)
+			(type default)
+		)
+	)
+	(wire
+		(pts
+			(xy 88.9 73.66) (xy 88.9 71.12)
 		)
 		(stroke
@@
 	(wire
 		(pts
-			(xy 86.36 66.04) (xy 86.36 73.66)
-		)
-		(stroke
-			(width 0)
-			(type default)
-		)
-	)
-	(wire
-		(pts
-			(xy 78.74 58.42) (xy 91.44 58.42)
-		)
-		(stroke
-			(width 0)
-			(type default)
-		)
-	)
-	(wire
-		(pts
-			(xy 93.98 71.12) (xy 124.46 71.12)
+			(xy 91.44 66.04) (xy 91.44 73.66)
+		)
+		(stroke
+			(width 0)
+			(type default)
+		)
+	)
+	(wire
+		(pts
+			(xy 78.74 58.42) (xy 83.82 58.42)
 		)
 		(stroke
@@
 	(wire
 		(pts
-			(xy 78.74 50.8) (xy 83.82 50.8)
+			(xy 78.74 50.8) (xy 81.28 50.8)
 		)
 		(stroke
@@
 	(wire
 		(pts
-			(xy 91.44 58.42) (xy 93.98 58.42)
-		)
-		(stroke
-			(width 0)
-			(type default)
-		)
-	)
-	(wire
-		(pts
-			(xy 93.98 73.66) (xy 93.98 71.12)
-		)
-		(stroke
-			(width 0)
-			(type default)
-		)
-	)
-	(wire
-		(pts
 			(xy 101.6 66.04) (xy 119.38 66.04)
 		)
@@
 	(wire
 		(pts
+			(xy 88.9 71.12) (xy 124.46 71.12)
+		)
+		(stroke
+			(width 0)
+			(type default)
+		)
+	)
+	(wire
+		(pts
 			(xy 129.54 63.5) (xy 124.46 63.5)
 		)
@@
 		(pts
 			(xy 127 60.96) (xy 127 55.88)
-		)
-		(stroke
-			(width 0)
-			(type default)
-		)
-	)
-	(wire
-		(pts
-			(xy 83.82 50.8) (xy 93.98 50.8)
 		)
 		(stroke
@@
 	(hierarchical_label "GND"
 		(shape bidirectional)
-		(at 88.9 86.36 270)
+		(at 86.36 86.36 270)
 		(effects
 			(font
@@
 	(symbol
 		(lib_id "RKL-Uncategorized:TPD4E02B04DQA")
-		(at 88.9 76.2 0)
+		(at 86.36 76.2 0)
 		(unit 1)
 		(exclude_from_sim no)
@@
 		(dnp no)
 		(property "Reference" "U5"
-			(at 78.74 78.74 0)
+			(at 76.2 78.74 0)
 			(effects
 				(font
@@
 		)
 		(property "Value" "TPD4E02B04DQA"
-			(at 73.66 81.28 0)
+			(at 71.12 81.28 0)
 			(effects
 				(font
@@
 		)
 		(property "Footprint" "Package_SON:USON-10_2.5x1.0mm_P0.5mm"
-			(at 88.9 76.2 0)
+			(at 86.36 76.2 0)
 			(effects
 				(font
@@
 		)
 		(property "Datasheet" "http://www.ti.com/lit/ds/symlink/tpd4e02b04.pdf"
-			(at 88.9 76.2 0)
+			(at 86.36 76.2 0)
 			(effects
 				(font
@@
 		)
 		(property "Description" ""
-			(at 88.9 76.2 0)
+			(at 86.36 76.2 0)
 			(effects
 				(font
@@
 		)
 		(property "LCSC" "C106794"
-			(at 88.9 76.2 0)
+			(at 86.36 76.2 0)
 			(effects
 				(font
@@
 		)
 		(property "Basic/Extended" "E"
-			(at 88.9 76.2 0)
+			(at 86.36 76.2 0)
 			(effects
 				(font
@@
 		)
 		(property "JLCPCB_CORRECTION" "0;0;-90"
-			(at 88.9 76.2 0)
-			(effects
-				(font
+			(at 86.36 76.2 0)
+			(effects
+				(font
