File: hw/ZakladniElektronika/HlavniDeska/charging.kicad_sch (KiCad schematic)
At the start: 16 parts, among them J1 Conn_01x02, U3 BQ25895M

Commit message: Hw wip
Parts:
- R19: value 330 -> 150; Basic/Extended B -> (none); LCSC C25104 -> (none); Price (100ks) 0.0005 -> (none); Price (1ks) 0.0005 -> (none)
Changed lines of the file:
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@@
 		(at 129.54 99.06)
 	)
+	(bus_entry
+		(at 114.3 93.98)
+		(size 2.54 -2.54)
+		(stroke
+			(width 0)
+			(type default)
+		)
+	)
+	(bus_entry
+		(at 114.3 88.9)
+		(size 2.54 -2.54)
+		(stroke
+			(width 0)
+			(type default)
+		)
+	)
+	(bus_entry
+		(at 114.3 71.12)
+		(size 2.54 -2.54)
+		(stroke
+			(width 0)
+			(type default)
+		)
+	)
+	(bus_entry
+		(at 114.3 73.66)
+		(size 2.54 -2.54)
+		(stroke
+			(width 0)
+			(type default)
+		)
+	)
+	(bus_entry
+		(at 114.3 91.44)
+		(size 2.54 -2.54)
+		(stroke
+			(width 0)
+			(type default)
+		)
+	)
+	(bus_entry
+		(at 114.3 73.66)
+		(size 2.54 -2.54)
+		(stroke
+			(width 0)
+			(type default)
+		)
+	)
+	(bus
+		(pts
+			(xy 114.3 76.2) (xy 101.6 76.2)
+		)
+		(stroke
+			(width 0)
+			(type default)
+		)
+	)
+	(bus
+		(pts
+			(xy 101.6 101.6) (xy 114.3 101.6)
+		)
+		(stroke
+			(width 0)
+			(type default)
+		)
+	)
 	(wire
 		(pts
@@
 		)
 	)
+	(bus
+		(pts
+			(xy 114.3 73.66) (xy 114.3 76.2)
+		)
+		(stroke
+			(width 0)
+			(type default)
+		)
+	)
 	(wire
 		(pts
@@
 		)
 	)
+	(bus
+		(pts
+			(xy 114.3 93.98) (xy 114.3 91.44)
+		)
+		(stroke
+			(width 0)
+			(type default)
+		)
+	)
 	(wire
 		(pts
@@
 	(wire
 		(pts
+			(xy 129.54 71.12) (xy 116.84 71.12)
+		)
+		(stroke
+			(width 0)
+			(type default)
+		)
+	)
+	(wire
+		(pts
 			(xy 121.92 101.6) (xy 121.92 76.2)
 		)
@@
 		)
 	)
+	(bus
+		(pts
+			(xy 114.3 71.12) (xy 114.3 73.66)
+		)
+		(stroke
+			(width 0)
+			(type default)
+		)
+	)
 	(wire
 		(pts
@@
 	(wire
 		(pts
+			(xy 116.84 86.36) (xy 129.54 86.36)
+		)
+		(stroke
+			(width 0)
+			(type default)
+		)
+	)
+	(wire
+		(pts
 			(xy 121.92 76.2) (xy 129.54 76.2)
 		)
@@
 		)
 	)
-	(wire
-		(pts
-			(xy 114.3 86.36) (xy 129.54 86.36)
-		)
-		(stroke
-			(width 0)
-			(type default)
-		)
-	)
-	(wire
-		(pts
-			(xy 114.3 91.44) (xy 129.54 91.44)
+	(bus
+		(pts
+			(xy 114.3 101.6) (xy 114.3 93.98)
 		)
 		(stroke
@@
 	(wire
 		(pts
+			(xy 129.54 68.58) (xy 116.84 68.58)
+		)
+		(stroke
+			(width 0)
+			(type default)
+		)
+	)
+	(wire
+		(pts
 			(xy 170.18 93.98) (xy 172.72 93.98)
 		)
@@
 		)
 	)
+	(bus
+		(pts
+			(xy 114.3 91.44) (xy 114.3 88.9)
+		)
+		(stroke
+			(width 0)
+			(type default)
+		)
+	)
 	(wire
 		(pts
@@
 	(wire
 		(pts
+			(xy 116.84 91.44) (xy 129.54 91.44)
+		)
+		(stroke
+			(width 0)
+			(type default)
+		)
+	)
+	(wire
+		(pts
 			(xy 149.86 91.44) (xy 152.4 91.44)
 		)
@@
 	(wire
 		(pts
-			(xy 114.3 88.9) (xy 129.54 88.9)
-		)
-		(stroke
-			(width 0)
-			(type default)
-		)
-	)
-	(wire
-		(pts
 			(xy 149.86 99.06) (xy 172.72 99.06)
 		)
@@
 	(wire
 		(pts
+			(xy 116.84 88.9) (xy 129.54 88.9)
+		)
+		(stroke
+			(width 0)
+			(type default)
+		)
+	)
+	(wire
+		(pts
 			(xy 152.4 68.58) (xy 154.94 68.58)
 		)
@@
 			(width 0)
 			(type default)
+		)
+	)
+	(label "D+"
+		(at 116.84 68.58 0)
+		(fields_autoplaced yes)
+		(effects
+			(font
+				(size 1.27 1.27)
+			)
+			(justify left bottom)
+		)
+	)
+	(label "SCL"
+		(at 116.84 88.9 0)
+		(effects
+			(font
+				(size 1.27 1.27)
+			)
+			(justify left bottom)
 		)
 	)
@@
 		)
 	)
+	(label "SDA"
+		(at 116.84 86.36 0)
+		(effects
+			(font
+				(size 1.27 1.27)
+			)
+			(justify left bottom)
+		)
+	)
 	(label "SYS"
 		(at 227.33 78.74 180)
@@
 			)
 			(justify right bottom)
+		)
+	)
+	(label "D-"
+		(at 116.84 71.12 0)
+		(fields_autoplaced yes)
+		(effects
+			(font
+				(size 1.27 1.27)
+			)
+			(justify left bottom)
+		)
+	)
+	(label "INT"
+		(at 116.84 91.44 0)
+		(effects
+			(font
+				(size 1.27 1.27)
+			)
+			(justify left bottom)
 		)
 	)
@@
 		)
 	)
-	(hierarchical_label "D-"
+	(hierarchical_label "{USB}"
 		(shape bidirectional)
-		(at 129.54 71.12 180)
+		(at 101.6 76.2 180)
+		(fields_autoplaced yes)
+		(effects
+			(font
+				(size 1.27 1.27)
+			)
+			(justify right)
+		)
+	)
+	(hierarchical_label "{I2C}"
+		(shape bidirectional)
+		(at 101.6 101.6 180)
 		(fields_autoplaced yes)
 		(effects
@@
 		)
 	)
-	(hierarchical_label "SCL"
-		(shape input)
-		(at 114.3 88.9 180)
-		(fields_autoplaced yes)
-		(effects
-			(font
-				(size 1.27 1.27)
-			)
-			(justify right)
-		)
-	)
 	(hierarchical_label "GND"
 		(shape bidirectional)
@@
 		)
 	)
-	(hierarchical_label "SDA"
-		(shape input)
-		(at 114.3 86.36 180)
-		(fields_autoplaced yes)
-		(effects
-			(font
-				(size 1.27 1.27)
-			)
-			(justify right)
-		)
-	)
 	(hierarchical_label "GND"
 		(shape bidirectional)
@@
 		(shape bidirectional)
 		(at 215.9 88.9 270)
-		(fields_autoplaced yes)
-		(effects
-			(font
-				(size 1.27 1.27)
-			)
-			(justify right)
-		)
-	)
-	(hierarchical_label "INT"
-		(shape input)
-		(at 114.3 91.44 180)
-		(fields_autoplaced yes)
-		(effects
-			(font
-				(size 1.27 1.27)
-			)
-			(justify right)
-		)
-	)
-	(hierarchical_label "D+"
-		(shape bidirectional)
-		(at 129.54 68.58 180)
 		(fields_autoplaced yes)
 		(effects
@@
 			)
 		)
-		(property "Value" "330"
+		(property "Value" "150"
 			(at 119.38 106.68 0)
 			(effects
@@
 			)
 		)
-		(property "Basic/Extended" "B"
+		(property "Basic/Extended" ""
 			(at 121.92 105.41 0)
 			(effects
@@
 			)
 		)
-		(property "LCSC" "C25104"
+		(property "LCSC" ""
 			(at 121.92 105.41 0)
 			(effects
@@
 			)
 		)
-		(property "Price (100ks)" "0.0005"
+		(property "Price (100ks)" ""
 			(at 121.92 105.41 0)
 			(effects
@@
 			)
 		)
-		(property "Price (1ks)" "0.0005"
+		(property "Price (1ks)" ""
 			(at 121.92 105.41 0)
 			(effects

Commit message: Hw PCB
Parts:
- removed D124: LED, LED_SMD:LED_0603_1608Metric, symbol Device:LED
- removed J1: Conn_01x02, Connector_PinSocket_2.54mm:PinSocket_1x02_P2.54mm_Vertical, symbol Connector_Generic:Conn_01x02
- removed R18: 56k, Resistor_SMD:R_0402_1005Metric, symbol Device:R
Connections:
- net CHARGER_STAT: now reaches U3.4 (STAT)
- net SW: now reaches C6.1, L6.1, U3.19 (SW), U3.20 (SW)

Commit message: Bordel Hw
Parts:
- R19: LCSC (none) -> C2909321
- U3: LCSC C485917 -> C80200
Connections:
- net GND: no longer U3.9 (~{CE})
- new net CE: U3.9 (~{CE})
Changed lines of the file:
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@@
-	)
-	(junction
-		(at 127 96.52)
-		(diameter 0)
-		(color 0 0 0 0)
 	)
 	(junction
@@
 	(wire
 		(pts
-			(xy 127 93.98) (xy 127 96.52)
+			(xy 127 93.98) (xy 127 109.22)
 		)
 		(stroke
@@
 	(wire
 		(pts
-			(xy 127 96.52) (xy 129.54 96.52)
-		)
-		(stroke
-			(width 0)
-			(type default)
-		)
-	)
-	(wire
-		(pts
 			(xy 205.74 81.28) (xy 203.2 81.28)
 		)
@@
 	(wire
 		(pts
-			(xy 127 96.52) (xy 127 109.22)
-		)
-		(stroke
-			(width 0)
-			(type default)
-		)
-	)
-	(wire
-		(pts
 			(xy 149.86 78.74) (xy 165.1 78.74)
 		)
@@
 		(pts
 			(xy 149.86 81.28) (xy 203.2 81.28)
+		)
+		(stroke
+			(width 0)
+			(type default)
+		)
+	)
+	(wire
+		(pts
+			(xy 119.38 96.52) (xy 129.54 96.52)
 		)
 		(stroke
@@
 		(shape bidirectional)
 		(at 160.02 109.22 270)
+		(effects
+			(font
+				(size 1.27 1.27)
+			)
+			(justify right)
+		)
+	)
+	(hierarchical_label "CE"
+		(shape input)
+		(at 119.38 96.52 180)
 		(effects
 			(font
@@
 			)
 		)
-		(property "LCSC" ""
+		(property "LCSC" "C2909321"
 			(at 121.92 105.41 0)
 			(effects
@@
 			)
 		)
-		(property "LCSC" "C485917"
+		(property "LCSC" "C80200"
 			(at 139.7 81.28 0)
 			(effects
