File: hw/ZakladniElektronika/HlavniDeska/multiplier.kicad_sch (KiCad schematic)
At the start: 23 parts, among them U10 NCP708, U16 TPS61088RHLR

Commit message: Hw wip
Other:
- moved on the sheet: C145, C152
Changed lines of the file:
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@@
+	)
+	(junction
+		(at 139.7 50.8)
+		(diameter 0)
+		(color 0 0 0 0)
 	)
 	(junction
@@
 	)
 	(junction
-		(at 72.39 50.8)
-		(diameter 0)
-		(color 0 0 0 0)
-	)
-	(junction
 		(at 78.74 104.14)
 		(diameter 0)
@@
 	)
 	(junction
-		(at 137.16 50.8)
+		(at 88.9 50.8)
 		(diameter 0)
 		(color 0 0 0 0)
@@
 	(wire
 		(pts
-			(xy 72.39 63.5) (xy 72.39 62.23)
+			(xy 88.9 63.5) (xy 88.9 62.23)
 		)
 		(stroke
@@
 	(wire
 		(pts
-			(xy 127 50.8) (xy 137.16 50.8)
+			(xy 139.7 50.8) (xy 161.29 50.8)
+		)
+		(stroke
+			(width 0)
+			(type default)
+		)
+	)
+	(wire
+		(pts
+			(xy 127 50.8) (xy 139.7 50.8)
 		)
 		(stroke
@@
 	(wire
 		(pts
-			(xy 137.16 50.8) (xy 161.29 50.8)
-		)
-		(stroke
-			(width 0)
-			(type default)
-		)
-	)
-	(wire
-		(pts
-			(xy 72.39 54.61) (xy 72.39 50.8)
+			(xy 88.9 54.61) (xy 88.9 50.8)
 		)
 		(stroke
@@
 	(wire
 		(pts
-			(xy 72.39 50.8) (xy 101.6 50.8)
-		)
-		(stroke
-			(width 0)
-			(type default)
-		)
-	)
-	(wire
-		(pts
 			(xy 97.79 124.46) (xy 97.79 132.08)
 		)
@@
 	(wire
 		(pts
-			(xy 53.34 50.8) (xy 72.39 50.8)
+			(xy 53.34 50.8) (xy 88.9 50.8)
 		)
 		(stroke
@@
 	(wire
 		(pts
-			(xy 137.16 50.8) (xy 137.16 52.07)
+			(xy 139.7 50.8) (xy 139.7 52.07)
 		)
 		(stroke
@@
 		(pts
 			(xy 127 104.14) (xy 127 99.06)
+		)
+		(stroke
+			(width 0)
+			(type default)
+		)
+	)
+	(wire
+		(pts
+			(xy 88.9 50.8) (xy 101.6 50.8)
 		)
 		(stroke
@@
 	(hierarchical_label "GND"
 		(shape bidirectional)
-		(at 137.16 59.69 270)
+		(at 139.7 59.69 270)
 		(fields_autoplaced yes)
 		(effects
@@
 	(hierarchical_label "GND"
 		(shape bidirectional)
-		(at 72.39 63.5 270)
+		(at 88.9 63.5 270)
 		(fields_autoplaced yes)
 		(effects
@@
 	(symbol
 		(lib_id "Device:C")
-		(at 137.16 55.88 0)
+		(at 139.7 55.88 0)
 		(unit 1)
 		(exclude_from_sim no)
@@
 		(fields_autoplaced yes)
 		(property "Reference" "C152"
-			(at 140.97 54.6099 0)
+			(at 143.51 54.6099 0)
 			(effects
 				(font
@@
 		)
 		(property "Value" "10u"
-			(at 140.97 57.1499 0)
+			(at 143.51 57.1499 0)
 			(effects
 				(font
@@
 		)
 		(property "Footprint" "Capacitor_SMD:C_0603_1608Metric"
-			(at 138.1252 59.69 0)
+			(at 140.6652 59.69 0)
 			(effects
 				(font
@@
 		)
 		(property "Datasheet" "~"
-			(at 137.16 55.88 0)
+			(at 139.7 55.88 0)
 			(effects
 				(font
@@
 		)
 		(property "Description" ""
-			(at 137.16 55.88 0)
+			(at 139.7 55.88 0)
 			(effects
 				(font
@@
 		)
 		(property "LCSC" "C96446"
-			(at 137.16 55.88 0)
+			(at 139.7 55.88 0)
 			(effects
 				(font
@@
 		)
 		(property "Basic/Extended" "B"
-			(at 137.16 55.88 0)
+			(at 139.7 55.88 0)
 			(effects
 				(font
@@
 		)
 		(property "info" "25V, X5R"
-			(at 137.16 55.88 0)
+			(at 139.7 55.88 0)
 			(effects
 				(font
@@
 	(symbol
 		(lib_id "Device:C")
-		(at 72.39 58.42 0)
+		(at 88.9 58.42 0)
 		(unit 1)
 		(exclude_from_sim no)
@@
 		(dnp no)
 		(property "Reference" "C145"
-			(at 75.311 57.2516 0)
+			(at 91.821 57.2516 0)
 			(effects
 				(font
@@
 		)
 		(property "Value" "4.7u"
-			(at 75.311 59.563 0)
+			(at 91.821 59.563 0)
 			(effects
 				(font
@@
 		)
 		(property "Footprint" "Capacitor_SMD:C_0603_1608Metric"
-			(at 73.3552 62.23 0)
+			(at 89.8652 62.23 0)
 			(effects
 				(font
@@
 		)
 		(property "Datasheet" "~"
-			(at 72.39 58.42 0)
+			(at 88.9 58.42 0)
 			(effects
 				(font
@@
 		)
 		(property "Description" ""
-			(at 72.39 58.42 0)
+			(at 88.9 58.42 0)
 			(effects
 				(font
@@
 		)
 		(property "LCSC" "C19666"
-			(at 72.39 58.42 0)
+			(at 88.9 58.42 0)
 			(effects
 				(font
@@
 		)
 		(property "Basic/Extended" "B"
-			(at 72.39 58.42 0)
+			(at 88.9 58.42 0)
 			(effects
 				(font
@@
 		)
 		(property "info" "16V, X5R"
-			(at 72.39 58.42 0)
-			(effects
-				(font
+			(at 88.9 58.42 0)
+			(effects
+				(font

Commit message: Bordel Hw
Parts:
- R58: LCSC C226818 -> C26957
Changed lines of the file:
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@@
 			)
 		)
-		(property "LCSC" "C226818"
+		(property "LCSC" "C26957"
 			(at 186.69 107.95 0)
 			(effects
