File: hw/ZakladniElektronika/HlavniDeska.kicad_sch (KiCad schematic)
At the start: 0 parts

Commit message: WIP
Parts:
- added BZ1: Buzzer, Robotarna_KiCad_Library:PKLCS1212E-(RH-Logic_piezzo), symbol Device:Buzzer
- added R23 (x2): 200, Resistor_SMD:R_0402_1005Metric, symbol Device:R
Connections:
- net ESP32S3/D+_ESP: now also R23.1
- net ESP32S3/D-_ESP: now also R23.1
- net ESP32S3/IO01: now also BZ1.2 (+)
- net ESP32S3/IO03-PD: now also BZ1.1 (-)
- new net ZpravceNapajeni/D+: R23.2
- new net ZpravceNapajeni/D-: R23.2
Other:
- added sheet GPSKomunikacniModul (HlavniDeska/GPSKomunikacniModul.kicad_sch)
- added sheet ModuloviKonektor (HlavniDeska/ModuloviKonektor.kicad_sch)
- sheet ZpravceNapajeni ports: added 1V8, 3V3, 5V, BUTTON_ON, CE, D+, D-, EN-5V, EN-ALL, GND, INT, ON, QON, SCL, SDA, VBUS, VCC; removed none

Commit message: Nastin schematu
Parts:
- removed R23 (x2): 200, Resistor_SMD:R_0402_1005Metric, symbol Device:R
Connections:
- no-connect marks 0 -> 2
Other:
- sheet ESP32S3 ports: added RST; removed none
- sheet ModuloviKonektor ports: added 5V, GND, INT, USART-RX, USART-TX; removed none
- moved on the sheet: BZ1

Commit message: Zaciame psat
Other:
- sheet ESP32S3 ports: added 5V-(programator); removed none
- sheet ZpravceNapajeni ports: added 5V-A, 5V-B, EN-5V-A, EN-5V-B; removed 5V, EN-5V
- moved on the sheet: BZ1

Commit message: WIP
Parts:
- added R5 (x3): 4.7k, Resistor_SMD:R_0201_0603Metric, symbol Device:R
Connections:
- net 3V3: now also R5.1, R5.1, R5.1
- net INT: now also R5.2
- net SCL: now also R5.2
- net SDA: now also R5.2

Commit message: Zavazbení zapínání
Other:
- sheet ModuloviKonektor renamed ModulovyKonektor
- sheet ZpravceNapajeni renamed SpravceNapajeni
- sheet ModulovyKonektor ports: added 3V3; removed none
Changed lines of the file:
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@@
+    (stroke (width 0) (type default))
+  )
+  (wire (pts (xy 71.12 127) (xy 86.36 127))
     (stroke (width 0) (type default))
   )
@@
     (stroke (width 0) (type default))
   )
+  (wire (pts (xy 86.36 60.96) (xy 109.22 60.96))
+    (stroke (width 0) (type default))
+  )
   (wire (pts (xy 134.62 152.4) (xy 134.62 147.32))
     (stroke (width 0.25) (type default) (color 0 0 0 1))
@@
   )
   (wire (pts (xy 175.26 128.27) (xy 195.58 128.27))
+    (stroke (width 0) (type default))
+  )
+  (wire (pts (xy 86.36 127) (xy 86.36 60.96))
     (stroke (width 0) (type default))
   )
@@
     (stroke (width 0.1524) (type solid))
     (fill (color 0 0 0 0.0000))
-    (property "Sheetname" "ModuloviKonektor" (at 38.1 125.73 0)
+    (property "Sheetname" "ModulovyKonektor" (at 38.1 125.73 0)
       (effects (font (size 2 2)) (justify left bottom))
     )
@@
     )
     (pin "USART-TX" input (at 71.12 137.16 0)
+      (effects (font (size 1.27 1.27)) (justify right))
+    )
+    (pin "3V3" input (at 71.12 127 0)
       (effects (font (size 1.27 1.27)) (justify right))
     )
@@
     (stroke (width 0.1524) (type solid))
     (fill (color 0 0 0 0.0000))
-    (property "Sheetname" "ZpravceNapajeni" (at 137.16 19.05 0)
+    (property "Sheetname" "SpravceNapajeni" (at 137.16 19.05 0)
       (effects (font (size 2 2)) (justify left bottom))
     )

Commit message: USB_multiplexer a přehlednost
Connections:
- no-connect marks 2 -> 0
Other:
- added sheet USBPřepínač (HlavniDeska/USBPrepinac.kicad_sch)
- sheet ESP32S3: file HlavniDeska/ESP332S3.kicad_sch -> HlavniDeska/ESP32S3.kicad_sch
- sheet ESP32S3 ports: added USB; removed D+_ESP, D-_ESP
- sheet GPSKomunikacniModul ports: added I2C, USB; removed SCL, SDA, USB_D+, USB_D-, WoWWAN(INT)
- sheet SpravceNapajeni ports: added DSEL, EN_ALL, I2C, USB; removed CE, D+, D-, EN-ALL, INT, QON, SCL, SDA
- sheet USB ports: added I2C, USB; removed D+_ESP, D-_ESP, INT, SCL, SDA
- moved on the sheet: BZ1, R5

Commit message: WIP
Changed lines of the file:
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@@
     (stroke (width 0) (type default))
   )
-  (bus (pts (xy 139.7 101.6) (xy 152.4 101.6))
+  (bus (pts (xy 139.7 101.6) (xy 165.1 101.6))
     (stroke (width 0) (type default))
   )
@@
     (stroke (width 0) (type default))
   )
-  (bus (pts (xy 165.1 101.6) (xy 215.9 101.6))
+  (bus (pts (xy 139.7 114.3) (xy 215.9 114.3))
     (stroke (width 0) (type default))
   )
@@
     (stroke (width 0) (type default))
   )
-  (bus (pts (xy 152.4 228.6) (xy 393.7 228.6))
+  (bus (pts (xy 165.1 228.6) (xy 393.7 228.6))
     (stroke (width 0) (type default))
   )
@@
     (stroke (width 0) (type default))
   )
-  (bus (pts (xy 152.4 127) (xy 152.4 228.6))
+  (bus (pts (xy 165.1 127) (xy 165.1 228.6))
     (stroke (width 0) (type default))
   )
@@
     (stroke (width 0.25) (type default) (color 0 0 0 1))
   )
-  (bus (pts (xy 152.4 101.6) (xy 152.4 50.8))
+  (bus (pts (xy 165.1 101.6) (xy 165.1 50.8))
     (stroke (width 0) (type default))
   )
   (bus (pts (xy 177.8 127) (xy 180.34 127))
-    (stroke (width 0) (type default))
-  )
-  (bus (pts (xy 165.1 114.3) (xy 165.1 101.6))
     (stroke (width 0) (type default))
   )
@@
     (stroke (width 0) (type default))
   )
-  (bus (pts (xy 139.7 114.3) (xy 165.1 114.3))
-    (stroke (width 0) (type default))
-  )
   (wire (pts (xy 35.56 215.9) (xy 35.56 139.7))
     (stroke (width 0.25) (type default) (color 0 0 0 1))
@@
     (stroke (width 0) (type default))
   )
-  (bus (pts (xy 139.7 127) (xy 152.4 127))
+  (bus (pts (xy 139.7 127) (xy 165.1 127))
     (stroke (width 0) (type default))
   )
@@
     (effects (font (size 1.27 1.27)) (justify right bottom))
   )
+  (label "I2C" (at 177.8 54.61 90) (fields_autoplaced)
+    (effects (font (size 1.27 1.27)) (justify left bottom))
+  )
   (label "INT" (at 214.63 139.7 180) (fields_autoplaced)
     (effects (font (size 1.27 1.27)) (justify right bottom))
   )
+  (label "USB-KomunikacniModul" (at 139.7 127 0) (fields_autoplaced)
+    (effects (font (size 1.27 1.27)) (justify left bottom))
+  )
   (label "SCL" (at 214.63 135.89 180) (fields_autoplaced)
     (effects (font (size 1.27 1.27)) (justify right bottom))
   )
+  (label "USB-C" (at 93.98 101.6 0) (fields_autoplaced)
+    (effects (font (size 1.27 1.27)) (justify left bottom))
+  )
   (label "KM_RXD" (at 280.67 116.84 0) (fields_autoplaced)
     (effects (font (size 1.27 1.27)) (justify left bottom))
   )
+  (label "USB-Nabijecka" (at 139.7 101.6 0) (fields_autoplaced)
+    (effects (font (size 1.27 1.27)) (justify left bottom))
+  )
+  (label "I2C" (at 177.8 127 0) (fields_autoplaced)
+    (effects (font (size 1.27 1.27)) (justify left bottom))
+  )
   (label "3V3" (at 77.47 167.64 0) (fields_autoplaced)
     (effects (font (size 1.27 1.27)) (justify left bottom))
   )
+  (label "I2C" (at 326.39 88.9 0) (fields_autoplaced)
+    (effects (font (size 1.27 1.27)) (justify left bottom))
+  )
+  (label "I2C" (at 76.2 127 0) (fields_autoplaced)
+    (effects (font (size 1.27 1.27)) (justify left bottom))
+  )
   (label "3V3" (at 209.55 78.74 0) (fields_autoplaced)
     (effects (font (size 1.27 1.27)) (justify left bottom))
@@
   )
   (label "KM_DTR" (at 280.67 124.46 0) (fields_autoplaced)
+    (effects (font (size 1.27 1.27)) (justify left bottom))
+  )
+  (label "USB-ESP" (at 139.7 114.3 0) (fields_autoplaced)
     (effects (font (size 1.27 1.27)) (justify left bottom))
   )
@@
     (effects (font (size 1.27 1.27)) (justify left))
   )
-  (hierarchical_label "5V" (shape input) (at 40.64 53.34 0) (fields_autoplaced)
+  (hierarchical_label "5V" (shape output) (at 40.64 53.34 0) (fields_autoplaced)
     (effects (font (size 1.27 1.27)) (justify left))
   )
@@
       (effects (font (size 1.27 1.27)) (justify left))
     )
-    (pin "5V-(programator)" input (at 215.9 76.2 180)
-      (effects (font (size 1.27 1.27)) (justify left))
-    )
-    (pin "USB" bidirectional (at 215.9 101.6 180)
+    (pin "5V-(programator)" output (at 215.9 76.2 180)
+      (effects (font (size 1.27 1.27)) (justify left))
+    )
+    (pin "USB" bidirectional (at 215.9 114.3 180)
       (effects (font (size 1.27 1.27)) (justify left))
     )
@@
       (effects (font (size 1.27 1.27)) (justify left))
     )
-    (pin "USB" bidirectional (at 152.4 50.8 270)
-      (effects (font (size 1.27 1.27)) (justify left))
-    )
+    (pin "USB" bidirectional (at 165.1 50.8 270)
+      (effects (font (size 1.27 1.27)) (justify left))
+    )

Commit message: Likvidace MiniUI jako samostatné desky a výběr všech komponent
Parts:
- added D126: green, LED_SMD:LED_0603_1608Metric, symbol Device:LED
- added D126: red, LED_SMD:LED_0603_1608Metric, symbol Device:LED
- added R13 (x2): 1k, Resistor_SMD:R_0402_1005Metric, symbol Device:R
- added SW1 (x2): SW_Push, RLK-ElectorMechanicalComponents:TCF2QR, symbol Switch:SW_Push
- BZ1: footprint Robotarna_KiCad_Library:PKLCS1212E-(RH-Logic_piezzo) -> RKL-StandardPackages:PKLCS1212E-(RH-Logic_piezzo); Basic/Extended (none) -> E
- R5: footprint Resistor_SMD:R_0201_0603Metric -> Resistor_SMD:R_0402_1005Metric; Basic/Extended E -> B; LCSC C270346 -> C25900
Connections:
- net GND: now also R13.1, R13.1, SW1.1, SW1.1
- new net: D126.1 (K), R13.2 (x2)
- new net ESP32S3/IO36: SW1.2
- new net ESP32S3/IO37: SW1.2
- new net ESP32S3/IO38: D126.2 (A)
- new net ESP32S3/IO39: D126.2 (A)
Other:
- sheet ESP32S3 ports: added none; removed BOOT, RST
- sheet SpravceNapajeni ports: added none; removed ON
- moved on the sheet: BZ1
