File: hw/ZakladniElektronika/HlavniDeska.kicad_sch (KiCad schematic)
At the start: 10 parts, among them SW1 SW_Push

Commit message: Výmněna ochrany baterie
Předchozí ochranný čip JLCPCB nemělo na skladě
Connections:
- no-connect marks 0 -> 3
Other:
- sheet ESP32S3 ports: added {USB}; removed 5V-(programator), USB
- sheet GPSKomunikacniModul ports: added {I2C}, {USB}; removed I2C, USB
- sheet SpravceNapajeni ports: added {I2C}, {USB}; removed I2C, USB
- sheet USB ports: added {I2C}, {USB}; removed I2C, USB
- sheet USBPřepínač ports: added 1{USB}, 2{USB}, 3{USB}, OUT{USB}; removed USB, USB1, USB2, USB3

Commit message: WIP
Changed lines of the file:
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@@
     (effects (font (size 1.27 1.27)) (justify right))
   )
-  (hierarchical_label "5V" (shape output) (at 40.64 53.34 0) (fields_autoplaced)
+  (hierarchical_label "5V-OUT" (shape output) (at 40.64 53.34 0) (fields_autoplaced)
     (effects (font (size 1.27 1.27)) (justify left))
   )

Commit message: PCB
Parts:
- removed D126: green, LED_SMD:LED_0603_1608Metric, symbol Device:LED
- removed D126: red, LED_SMD:LED_0603_1608Metric, symbol Device:LED
- added D121: LED_Dual_AKAK, RKL-LED:SMD,1.5x3.2mm 4pin, symbol Device:LED_Dual_AKAK
Connections:
- net ESP32S3/IO38: now also D121.3 (A2)
- net ESP32S3/IO39: now also D121.1 (A1)
- net at R13.2: now also D121.2 (K1)
- net at R13.2: now also D121.4 (K2)
Other:
- sheet USB ports: added VBUS; removed VUSB
- moved on the sheet: R13, SW1

Commit message: Řešení issue "Držák baterek" a " SemiSemafor V0"
Parts:
- BZ1: footprint RKL-StandardPackages:PKLCS1212E-(RH-Logic_piezzo) -> RKL-Audio:PKLCS1212E-(RH-Logic_piezzo)
Changed lines of the file:
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@@
       (effects (font (size 1.27 1.27)))
     )
-    (property "Footprint" "RKL-StandardPackages:PKLCS1212E-(RH-Logic_piezzo)" (at 283.845 165.1 90)
+    (property "Footprint" "RKL-Audio:PKLCS1212E-(RH-Logic_piezzo)" (at 283.845 165.1 90)
       (effects (font (size 1.27 1.27)) hide)
     )

Commit message: KiCad V8
Parts:
- renumbered R13 to R27, R13 to R28, R5 to R37, R5 to R38, R5 to R39, SW1 to SW2

Commit message: Hw wip
Connections:
- no-connect marks 3 -> 14
Other:
- removed sheet GPSKomunikacniModul
- sheet SpravceNapajeni ports: added OFF, USB_SEL, VUSB; removed 1V8, DSEL, EN_ALL, VBUS, VCC
- sheet USBPřepínač ports: added none; removed 3{USB}
- moved on the sheet: BZ1, D121, R27, R28, R37, R38, R39, SW1, SW2

Commit message: Hw PCB
Parts:
- removed D121: LED_Dual_AKAK, RKL-LED:SMD,1.5x3.2mm 4pin, symbol Device:LED_Dual_AKAK
- removed R27: 1k, Resistor_SMD:R_0402_1005Metric, symbol Device:R
- added C136, C137: 10uF, Capacitor_SMD:C_0603_1608Metric, symbol Device:C
- added D125: LED_ARGB, RKL-LED:XL-3806RGBC-4L, symbol Device:LED_ARGB
- added J1: Conn_02x09_Counter_Clockwise, Connector_PinHeader_2.54mm:PinHeader_2x09_P2.54mm_Vertical, symbol Connector_Generic:Conn_02x09_Odd_Even
- added J5: Micro_SD_Card, Connector_Card:microSD_HC_Molex_47219-2001, symbol Connector:Micro_SD_Card
- added R11, R5: 1k, Resistor_SMD:R_0402_1005Metric, symbol Device:R
- added R12, R13, R35, R36, R41: 10k, Resistor_SMD:R_0402_1005Metric, symbol Device:R
Connections:
- net 3V3: now also C136.1, C137.1, D125.1 (A), J5.4 (VDD), R35.1, R36.1, R41.1
- net ESP32S3/IO01: now also J1.1 (Pin_1); no longer BZ1.2 (+)
- net ESP32S3/IO02: now also J1.3 (Pin_3)
- net ESP32S3/IO03-PD: now also J5.2 (DAT3/CD); no longer BZ1.1 (-)
- net ESP32S3/IO10: now also R28.2, R13.2
- net ESP32S3/IO11: now also J5.3 (CMD), R41.2
- net ESP32S3/IO12: now also J5.5 (CLK), R36.2
- net ESP32S3/IO13: now also J5.7 (DAT0), R35.2
- net ESP32S3/IO14: now also J1.5 (Pin_5)
- net ESP32S3/IO15: now also BZ1.1 (-)
- net ESP32S3/IO16: now also BZ1.2 (+)
- net ESP32S3/IO17: now also J1.7 (Pin_7)
- net ESP32S3/IO18: now also J1.9 (Pin_9)
- net ESP32S3/IO38: now also R11.2, R12.1
- net ESP32S3/IO39: now also R5.2
- net ESP32S3/IO41: now also J1.11 (Pin_11)
- net ESP32S3/IO42: now also J1.13 (Pin_13)
- net ESP32S3/IO47: now also J1.15 (Pin_15)
- net ESP32S3/IO48: now also J1.17 (Pin_17)
- net GND: now also C136.2, C137.2, J1.10 (Pin_10), J1.12 (Pin_12), J1.14 (Pin_14), J1.16 (Pin_16), J1.18 (Pin_18), J1.2 (Pin_2), J1.4 (Pin_4), J1.6 (Pin_6), J1.8 (Pin_8), J5.6 (VSS), J5.9 (SHIELD), R12.2; no longer R28.1
- new net: D125.4 (BK), R28.1
- new net: D125.2 (RK), R11.1
- new net: D125.3 (GK), R5.1
- new net SpravceNapajeni/CHARGER_STAT: R13.1
- no-connect marks 14 -> 2
Other:
- sheet SpravceNapajeni ports: added CHARGER_STAT; removed none
- sheet USB ports: added none; removed {I2C}
- sheet USBPřepínač ports: added 0{USB}, USB_SEL, VUSB; removed 3V3, OUT{USB}, SEL0
- moved on the sheet: BZ1, R28, R37, R38, R39

Commit message: Bordel Hw
Parts:
- added R14, R15: 330, Resistor_SMD:R_0402_1005Metric, symbol Device:R
- added R16, R17: 10k, Resistor_SMD:R_0402_1005Metric, symbol Device:R
- BZ1: footprint RKL-Audio:PKLCS1212E-(RH-Logic_piezzo) -> RKL-Audio:ELKS-PIEZO; Basic/Extended E -> (none); LCSC C113159 -> C201041
- SW1, SW2: LCSC C240292 -> C495937
Connections:
- net 3V3: now also R16.1, R17.1
- net ESP32S3/IO15: now also R14.1; no longer BZ1.1 (-)
- net ESP32S3/IO16: now also R15.1; no longer BZ1.2 (+)
- net ESP32S3/IO36: now also R16.2
- net ESP32S3/IO37: now also R17.2
- new net: BZ1.1 (-), R14.2
- new net: BZ1.2 (+), R15.2
