File: hw/ZakladniElektronika/LedDeska/LedRing.kicad_sch (KiCad schematic)
At the start: 120 parts

Commit message: WIP
Parts:
- C12, C13, C14, C15, C16, C17, C18, C19, C20, C21, C22, C23, C24, C25, C26, C27, C28, C29, C30, C31, C32, C33, C34, C35, C36, C37, C38, C39, C40, C41, C42, C43, C44, C45, C46, C47, C48, C49, C50, C51, C52, C53, C54, C55, C56, C57, C58, C59, C60, C61, C62, C63, C64, C65, C66, C67, C68, C69, C70, C71: Basic/Extended (none) -> B; LCSC (none) -> C307331; info (none) -> 50V, X7R
Other:
- moved on the sheet: C12, C13, C14, C15, C16, C17, C18, C19, C20, C21, C22, C23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

Commit message: Likvidace MiniUI jako samostatné desky a výběr všech komponent
Parts:
- D1, D10, D11, D12, D13, D14, D15, D16, D17, D18, D19, D2, D20, D21, D22, D23, D24, D25, D26, D27, D28, D29, D3, D30, D31, D32, D33, D34, D35, D36, D37, D38, D39, D4, D40, D41, D42, D43, D44, D45, D46, D47, D48, D49, D5, D50, D51, D52, D53, D54, D55, D56, D57, D58, D59, D6, D60, D7, D8, D9: footprint RB3203-Lib:WS2812 -> RKL-LED:3528RGBW-WS2812B; Basic/Extended (none) -> E; LCSC (none) -> C2890364

Commit message: PCB
Connections:
- net at D54.4 (DIN): now also D53.2 (DOUT); no longer D48.2 (DOUT)
- net at D48.4 (DIN): now also D47.2 (DOUT); no longer D42.2 (DOUT)
- net at D52.2 (DOUT): now also D53.4 (DIN); no longer D58.4 (DIN)
- net at D46.2 (DOUT): now also D47.4 (DIN); no longer D52.4 (DIN)
- net at D54.2 (DOUT): now also D55.4 (DIN); no longer D60.4 (DIN)
- net at D49.2 (DOUT): now also D50.4 (DIN); no longer D55.4 (DIN)
- net at D49.4 (DIN): now also D48.2 (DOUT); no longer D43.2 (DOUT)
- net at D22.2 (DOUT): now also D23.4 (DIN); no longer D28.4 (DIN)
- net at D16.2 (DOUT): now also D17.4 (DIN); no longer D22.4 (DIN)
- net at D11.2 (DOUT): now also D12.4 (DIN); no longer D17.4 (DIN)
- net at D11.4 (DIN): now also D10.2 (DOUT); no longer D5.2 (DOUT)
- net at D41.2 (DOUT): now also D42.4 (DIN); no longer D47.4 (DIN)
- net at D26.4 (DIN): now also D25.2 (DOUT); no longer D20.2 (DOUT)
- net at D14.2 (DOUT): now also D15.4 (DIN); no longer D20.4 (DIN)
- net at D51.4 (DIN): now also D50.2 (DOUT); no longer D45.2 (DOUT)
- net at D39.2 (DOUT): now also D40.4 (DIN); no longer D45.4 (DIN)
- net at D3.2 (DOUT): now also D4.4 (DIN); no longer D9.4 (DIN)
- net at D3.4 (DIN): now also D2.2 (DOUT); no longer D56.2 (DOUT)
- net at D8.2 (DOUT): now also D9.4 (DIN); no longer D14.4 (DIN)
- net at D8.4 (DIN): now also D7.2 (DOUT); no longer D2.2 (DOUT)
- net at D34.4 (DIN): now also D33.2 (DOUT); no longer D28.2 (DOUT)
- net at D15.2 (DOUT): now also D16.4 (DIN); no longer D21.4 (DIN)
- net at D9.2 (DOUT): now also D10.4 (DIN); no longer D15.4 (DIN)
- net at D19.4 (DIN): now also D18.2 (DOUT); no longer D13.2 (DOUT)
- net at D13.4 (DIN): now also D12.2 (DOUT); no longer D7.2 (DOUT)
- net at D33.4 (DIN): now also D32.2 (DOUT); no longer D27.2 (DOUT)
- net at D27.4 (DIN): now also D26.2 (DOUT); no longer D21.2 (DOUT)
- net at D6.2 (DOUT): now also D7.4 (DIN); no longer D12.4 (DIN)
- net at D6.4 (DIN): now also D5.2 (DOUT); no longer D59.2 (DOUT)
- net at D56.4 (DIN): now also D55.2 (DOUT); no longer D50.2 (DOUT)
- net at D44.2 (DOUT): now also D45.4 (DIN); no longer D50.4 (DIN)
- net at D17.2 (DOUT): now also D18.4 (DIN); no longer D23.4 (DIN)
- net at D31.2 (DOUT): now also D32.4 (DIN); no longer D37.4 (DIN)
- net at D31.4 (DIN): now also D30.2 (DOUT); no longer D25.2 (DOUT)
- net at D43.4 (DIN): now also D42.2 (DOUT); no longer D37.2 (DOUT)
- net at D1.2 (DOUT): now also D2.4 (DIN); no longer D7.4 (DIN)
- net at D29.2 (DOUT): now also D30.4 (DIN); no longer D35.4 (DIN)
- net at D23.2 (DOUT): now also D24.4 (DIN); no longer D29.4 (DIN)
- net at D38.2 (DOUT): now also D39.4 (DIN); no longer D44.4 (DIN)
- net at D38.4 (DIN): now also D37.2 (DOUT); no longer D32.2 (DOUT)
- net at D51.2 (DOUT): now also D52.4 (DIN); no longer D57.4 (DIN)
- net at D36.4 (DIN): now also D35.2 (DOUT); no longer D30.2 (DOUT)
- net at D24.2 (DOUT): now also D25.4 (DIN); no longer D30.4 (DIN)
- net at D5.4 (DIN): now also D4.2 (DOUT); no longer D58.2 (DOUT)
- net at D34.2 (DOUT): now also D35.4 (DIN); no longer D40.4 (DIN)
- net at D41.4 (DIN): now also D40.2 (DOUT); no longer D35.2 (DOUT)
- net at D36.2 (DOUT): now also D37.4 (DIN); no longer D42.4 (DIN)
- net at D57.2 (DOUT): now also D58.4 (DIN); no longer D4.4 (DIN)
- net at D19.2 (DOUT): now also D20.4 (DIN); no longer D25.4 (DIN)
- net at D59.4 (DIN): now also D58.2 (DOUT); no longer D53.2 (DOUT)
- net at D46.4 (DIN): now also D45.2 (DOUT); no longer D40.2 (DOUT)
- new net: D20.2 (DOUT), D21.4 (DIN)
- new net: D28.2 (DOUT), D29.4 (DIN)
- new net: D59.2 (DOUT), D60.4 (DIN)
- new net: D27.2 (DOUT), D28.4 (DIN)
- new net: D13.2 (DOUT), D14.4 (DIN)
- new net: D43.2 (DOUT), D44.4 (DIN)
- new net: D56.2 (DOUT), D57.4 (DIN)
- new net: D21.2 (DOUT), D22.4 (DIN)

Commit message: Hw wip
Parts:
- renumbered C62 to C100, C68 to C101, C15 to C102, C21 to C103, C27 to C104, C33 to C105, C39 to C106, C45 to C107, C51 to C108, C57 to C109, C63 to C110, C69 to C111, C16 to C112, C22 to C113, C28 to C114, C34 to C115, C40 to C116, C46 to C117, C52 to C118, C58 to C119, C64 to C120, C70 to C121, C17 to C122, C23 to C123, C29 to C124, C35 to C125, C41 to C126, C47 to C127, C53 to C128, C59 to C129, C65 to C130, C71 to C131, C12 to C72, C18 to C73, C24 to C74, C30 to C75, C36 to C76, C42 to C77, C48 to C78, C54 to C79, C60 to C80, C66 to C81, C13 to C82, C19 to C83, C25 to C84, C31 to C85, C37 to C86, C43 to C87, C49 to C88, C55 to C89, C61 to C90, C67 to C91, C14 to C92, C20 to C93, C26 to C94, C32 to C95, C38 to C96, C44 to C97, C50 to C98, C56 to C99, D40 to D100, D41 to D101, D42 to D102, D43 to D103, D44 to D104, D45 to D105, D46 to D106, D47 to D107, D48 to D108, D49 to D109, D50 to D110, D51 to D111, D52 to D112, D53 to D113, D54 to D114, D55 to D115, D56 to D116, D57 to D117, D58 to D118, D59 to D119, D60 to D120, D1 to D61, D2 to D62, D3 to D63, D4 to D64, D5 to D65, D6 to D66, D7 to D67, D8 to D68, D9 to D69, D10 to D70, D11 to D71, D12 to D72, D13 to D73, D14 to D74, D15 to D75, D16 to D76, D17 to D77, D18 to D78, D19 to D79, D20 to D80, D21 to D81, D22 to D82, D23 to D83, D24 to D84, D25 to D85, D26 to D86, D27 to D87, D28 to D88, D29 to D89, D30 to D90, D31 to D91, D32 to D92, D33 to D93, D34 to D94, D35 to D95, D36 to D96, D37 to D97, D38 to D98, D39 to D99
