File: text/text/PraktickaCast/sch/power_manager.kicad_sch (KiCad schematic)
At the start: 32 parts, among them Q1 NMOS, Q2 NMOS, Q3 NMOS, Q4 NMOS, Q5 NMOS, Q6 NMOS, Q7 NMOS, Q8 NMOS, SW1 OFF, SW2 ON, SW3 OFF, U1 SL8261D-G3JE, U2 SL8261D-G3JE

Commit message: Text WIP
Parts:
- removed Qp1, Qp2: JMTV210P02A, Package_DFN_QFN:Diodes_UDFN2020-6_Type-F, symbol RKL-MOSFET:JMTV210P02A
- removed SW3: OFF, Button_Switch_SMD:SW_Push_1P1T_NO_Vertical_Wuerth_434133025816, symbol Switch:SW_Push
- added D1: LED, symbol Device:LED
- added D122: D_Dual_CommonCathode_AAK_Parallel, Package_TO_SOT_SMD:SOT-723, symbol Device:D_Dual_CommonCathode_AAK_Parallel
- added D125: LED_ARGB, RKL-LED:XL-3806RGBC-4L, symbol Device:LED_ARGB
- added Q10, Q9: NMOS, Package_TO_SOT_SMD:SOT-723, symbol Device:Q_NMOS_GSD
- added Q11: BC547, Package_TO_SOT_THT:TO-92_Inline, symbol Transistor_BJT:BC547
- added Q12: BC557, Package_TO_SOT_THT:TO-92_Inline, symbol Transistor_BJT:BC557
- added Qp1, Qp2, Qp3, Qp4: JMTV210P02A, symbol Simulation_SPICE:PMOS
- added R15, R16, R19, R32: 10k, Resistor_SMD:R_0402_1005Metric, symbol Device:R
- added R17, R18, R28: 1k, Resistor_SMD:R_0402_1005Metric, symbol Device:R
- added R20: 1k - 22k, symbol Device:R
- added R21: 6k7 - 54k, symbol Device:R
- added R22: 28k - 220k, symbol Device:R
Connections:
- net 3V3: now also D125.1 (A)
- net Baterie: now also Qp1.3 (S), Qp2.3 (S)
- net GND: now also D1.1 (K), Q10.2 (S), Q11.3 (E), Q9.2 (S), R19.2
- net Napájení zeřízení: now also Qp1.1 (D), Qp2.1 (D)
- net at Q4.3 (D), Q6.3 (D), R11.2: now also Qp2.2 (G)
- net at Q2.3 (D), R2.2: now also Qp1.2 (G)
- new net: Q9.3 (D), Qp3.2 (G), R15.2
- new net: D125.4 (BK), R28.1
- new net: D125.2 (RK), R18.1
- new net: D125.3 (GK), R17.1
- new net: Q11.2 (B), R21.2
- new net: Q10.3 (D), Qp4.2 (G), R32.2
- new net: Q11.1 (C), R20.2, R22.1
- new net: D1.2 (A), Q12.1 (C)
- new net: Q12.2 (B), R22.2
- new net +12V: Q12.3 (E), R20.1
- new net 5V-A: Qp3.1 (D)
- new net 5V-B: Qp4.1 (D)
- new net 5V-IN: Qp3.3 (S), Qp4.3 (S), R15.1, R32.1
- new net CHARGER_STAT: R16.2
- new net EN-5V-A: D122.1 (K), Q9.1 (G)
- new net EN-5V-B: D122.2 (K), Q10.1 (G)
- new net IO10: R16.1, R28.2
- new net IO38: R18.2, R19.1
- new net IO39: R17.2
- new net Power multiplier/EN-5V: D122.3 (A)
Other:
- added sheet Power multiplier (multiplier.kicad_sch)
- note added: "ESP"
- moved on the sheet: C2, C3, Q1, Q2, Q3, Q4, Q5, Q6, Q7, Q8, R10, R11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
